File: EAGLE/project/473/nucleum.sch (EAGLE design)
At the start: 40 parts, among them J1 TC2030-JLINK-NL, J2 SH_MALE_2/1MM, J3 ATUM-HEADER, U1 FM25L04B-DG, U3 RV-3049-C3, U4 TPS62740, U5 NRF51822QF, X1 EPSON-FA-128, X2 ABS05-32.768KHZ-T

Commit message: changed to sheet 2 test
Other:
- note added: "Sup"
- moved on the sheet: C16, U4
Changed lines of the file:
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@@
 <?xml version="1.0" encoding="utf-8"?>
 <!DOCTYPE eagle SYSTEM "eagle.dtd">
-<eagle version="6.5.0">
+<eagle version="6.6.0">
 <drawing>
 <settings>
@@
 <plain>
 <text x="91.44" y="127" size="1.778" layer="98">A-1.8V B-3.0V Output</text>
+<text x="35.56" y="76.2" size="1.778" layer="91">Sup</text>
 </plain>
 <instances>
 <instance part="FRAME2" gate="G$1" x="0" y="0"/>
 <instance part="FRAME2" gate="G$2" x="147.32" y="0"/>
-<instance part="U4" gate="G$1" x="86.36" y="109.22"/>
+<instance part="U4" gate="G$1" x="86.36" y="142.24"/>
 <instance part="GND2" gate="1" x="71.12" y="93.98"/>
 <instance part="GND6" gate="1" x="104.14" y="93.98"/>
@@
 <attribute name="DIGIKEY" x="43.18" y="114.3" size="1.27" layer="96" display="off"/>
 </instance>
-<instance part="C16" gate="G$1" x="109.22" y="111.76" smashed="yes">
-<attribute name="DIGIKEY" x="109.22" y="111.76" size="1.27" layer="96" display="off"/>
-<attribute name="NAME" x="106.68" y="110.49" size="1.778" layer="95" ratio="12" rot="R90" align="bottom-center"/>
-<attribute name="VALUE" x="111.76" y="110.49" size="1.778" layer="96" ratio="12" rot="R270" align="bottom-center"/>
+<instance part="C16" gate="G$1" x="119.38" y="96.52" smashed="yes">
+<attribute name="DIGIKEY" x="119.38" y="96.52" size="1.27" layer="96" display="off"/>
+<attribute name="NAME" x="116.84" y="95.25" size="1.778" layer="95" ratio="12" rot="R90" align="bottom-center"/>
+<attribute name="VALUE" x="121.92" y="95.25" size="1.778" layer="96" ratio="12" rot="R270" align="bottom-center"/>
 </instance>
 <instance part="J2" gate="G$1" x="175.26" y="114.3" rot="R180"/>
@@
 <wire x1="71.12" y1="96.52" x2="71.12" y2="99.06" width="0.1524" layer="91"/>
 <pinref part="U4" gate="G$1" pin="GND"/>
-<wire x1="71.12" y1="99.06" x2="73.66" y2="99.06" width="0.1524" layer="91"/>
+<wire x1="71.12" y1="99.06" x2="73.66" y2="132.08" width="0.1524" layer="91"/>
 <wire x1="43.18" y1="109.22" x2="43.18" y2="99.06" width="0.1524" layer="91"/>
 <wire x1="43.18" y1="99.06" x2="48.26" y2="99.06" width="0.1524" layer="91"/>
@@
 <pinref part="U4" gate="G$1" pin="VSEL1"/>
 <wire x1="48.26" y1="99.06" x2="71.12" y2="99.06" width="0.1524" layer="91"/>
-<wire x1="73.66" y1="111.76" x2="71.12" y2="111.76" width="0.1524" layer="91"/>
+<wire x1="73.66" y1="144.78" x2="71.12" y2="111.76" width="0.1524" layer="91"/>
 <wire x1="71.12" y1="111.76" x2="71.12" y2="109.22" width="0.1524" layer="91"/>
 <pinref part="C15" gate="G$1" pin="2"/>
 <pinref part="U4" gate="G$1" pin="VSEL2"/>
 <wire x1="71.12" y1="109.22" x2="71.12" y2="99.06" width="0.1524" layer="91"/>
-<wire x1="73.66" y1="109.22" x2="71.12" y2="109.22" width="0.1524" layer="91"/>
+<wire x1="73.66" y1="142.24" x2="71.12" y2="109.22" width="0.1524" layer="91"/>
 <junction x="71.12" y="109.22"/>
 <pinref part="S1" gate="G$1" pin="A"/>
@@
 <segment>
 <pinref part="U4" gate="G$1" pin="CTRL"/>
-<wire x1="99.06" y1="101.6" x2="104.14" y2="101.6" width="0.1524" layer="91"/>
+<wire x1="99.06" y1="134.62" x2="104.14" y2="101.6" width="0.1524" layer="91"/>
 <wire x1="104.14" y1="101.6" x2="104.14" y2="96.52" width="0.1524" layer="91"/>
 <pinref part="GND6" gate="1" pin="GND"/>
 <wire x1="104.14" y1="101.6" x2="109.22" y2="101.6" width="0.1524" layer="91"/>
-<wire x1="109.22" y1="101.6" x2="109.22" y2="106.68" width="0.1524" layer="91"/>
+<wire x1="109.22" y1="101.6" x2="119.38" y2="91.44" width="0.1524" layer="91"/>
 <junction x="104.14" y="101.6"/>
 <pinref part="C16" gate="G$1" pin="2"/>
@@
 <pinref part="U4" gate="G$1" pin="VOUT"/>
 <wire x1="119.38" y1="116.84" x2="109.22" y2="116.84" width="0.1524" layer="91"/>
-<wire x1="109.22" y1="116.84" x2="99.06" y2="116.84" width="0.1524" layer="91"/>
-<wire x1="109.22" y1="114.3" x2="109.22" y2="116.84" width="0.1524" layer="91"/>
+<wire x1="109.22" y1="116.84" x2="99.06" y2="149.86" width="0.1524" layer="91"/>
+<wire x1="119.38" y1="99.06" x2="109.22" y2="116.84" width="0.1524" layer="91"/>
 <junction x="109.22" y="116.84"/>
 <junction x="119.38" y="119.38"/>
@@
 <segment>
 <pinref part="U4" gate="G$1" pin="VIN"/>
-<wire x1="73.66" y1="119.38" x2="71.12" y2="119.38" width="0.1524" layer="91"/>
+<wire x1="73.66" y1="152.4" x2="71.12" y2="119.38" width="0.1524" layer="91"/>
 <wire x1="71.12" y1="119.38" x2="48.26" y2="119.38" width="0.1524" layer="91"/>
 <wire x1="48.26" y1="119.38" x2="43.18" y2="119.38" width="0.1524" layer="91"/>
 <wire x1="43.18" y1="119.38" x2="43.18" y2="116.84" width="0.1524" layer="91"/>
 <pinref part="U4" gate="G$1" pin="EN"/>
-<wire x1="73.66" y1="116.84" x2="71.12" y2="116.84" width="0.1524" layer="91"/>
+<wire x1="73.66" y1="149.86" x2="71.12" y2="116.84" width="0.1524" layer="91"/>
 <wire x1="71.12" y1="116.84" x2="71.12" y2="119.38" width="0.1524" layer="91"/>
 <junction x="71.12" y="119.38"/>
@@
 <pinref part="U4" gate="G$1" pin="SW"/>
 <pinref part="L2" gate="G$1" pin="1"/>
-<wire x1="99.06" y1="119.38" x2="101.6" y2="119.38" width="0.1524" layer="91"/>
+<wire x1="99.06" y1="152.4" x2="101.6" y2="119.38" width="0.1524" layer="91"/>
 </segment>
 </net>
@@
 <segment>
 <pinref part="U4" gate="G$1" pin="VSEL4"/>
-<wire x1="73.66" y1="104.14" x2="68.58" y2="104.14" width="0.1524" layer="91"/>
+<wire x1="73.66" y1="137.16" x2="68.58" y2="104.14" width="0.1524" layer="91"/>
 <pinref part="U4" gate="G$1" pin="VSEL3"/>
 <wire x1="68.58" y1="104.14" x2="60.96" y2="104.14" width="0.1524" layer="91"/>
-<wire x1="73.66" y1="106.68" x2="68.58" y2="106.68" width="0.1524" layer="91"/>
+<wire x1="73.66" y1="139.7" x2="68.58" y2="106.68" width="0.1524" layer="91"/>
 <wire x1="68.58" y1="106.68" x2="68.58" y2="104.14" width="0.1524" layer="91"/>
 <junction x="68.58" y="104.14"/>
