File: EAGLE/project/473/nucleum.sch (EAGLE design)
At the start: 40 parts, among them J1 TC2030-JLINK-NL, J2 SH_MALE_2/1MM, J3 ATUM-HEADER, U1 FM25L04B-DG, U3 RV-3049-C3, U4 TPS62740, U5 NRF51822QF, X1 EPSON-FA-128, X2 ABS05-32.768KHZ-T

Commit message: PCB Schematic
Parts:
- added C17: 0.1µF, microbuilder:CAP_CERAMIC_0805
- added C18, C19: 1µF, microbuilder:CAP_CERAMIC_0805
- added C20, C21: 10µF, microbuilder:CAP_CERAMIC_0805
- added C22, C24: 0.1uF, SparkFun:CAP0603-CAP
- added C23: 2.2nF, SparkFun:CAP0603-CAP
- added C25: 10nF, SparkFun:CAP0603-CAP
- added FB1, FB2: (no value), microbuilder:FERRITE_0805
- added FID1, FID2, FID3: FIDUCIAL"", microbuilder:FIDUCIAL""
- added FRAME4: FRAME-LETTER, SparkFun-Aesthetics:FRAME-LETTER
- added IC1: LS013B4DN04, microbuilder:SHARP_MEMORYLCD_10PIN
- added JP1: (no value), microbuilder:HEADER-1X970MIL
- added JP2, JP5: FIDUCIALUFIDUCIAL, SparkFun:FIDUCIALUFIDUCIAL
- added JP3, JP4: STAND-OFFTIGHT, SparkFun:STAND-OFFTIGHT
- added JP6: M10", SparkFun:M10"
- added R10, R11: 10k, SparkFun:RESISTOR0603-RES
- added R7, R8, R9: 10K, microbuilder:RESISTOR_0805
- added SJ1: (no value), SparkFun:SOLDERJUMPER_2WAYPASTE2&3
- added SJ2, SJ3: SOLDERJUMPERTRACE, SparkFun:SOLDERJUMPERTRACE
- added U$21, U$22, U$27, U$28: MOUNTINGHOLE3.0THIN, microbuilder:MOUNTINGHOLE3.0THIN
- added U$30: OSHW-LOGOS, SparkFun:OSHW-LOGOS
- added U$31: REVISION, SparkFun-Aesthetics:REVISION
- added U2: 74HC4050D, microbuilder:74HC4050D
- added U6: MCP1824T-3302E/OT, microbuilder:VREG_SOT23-5
- added U7: MPU-6050-1, Testing:MPU-6050-1
Connections:
- new net 3.3V: C19.P$1, C21.P$1, FB1.P$1, IC1.VDD, JP1.2, R7.1, U2.VCC, U6.OUT
- new net ADO: SJ1.2, U7.AD0
- new net AGND: C18.P$2, FB2.P$2, IC1.VSSA
- new net AUX_SCL: JP6.2, U7.AUX_CL
- new net AUX_SDA: JP6.1, U7.AUX_DA
- new net AVDD: C18.P$1, FB1.P$2, IC1.VDDA
- new net CLKIN: JP6.3, SJ2.2, U7.CLKIN
- new net DISP: C17.P$1, IC1.DISP, U2.5Y
- new net DISP_5V: JP1.8, R7.2, U2.5A
- new net EXTCOMIN: IC1.EXTCOMIN, U2.4Y
- new net EXTCOMIN_5V: JP1.9, R8.1, U2.4A
- new net EXTMODE: IC1.EXTMODE, U2.6Y
- new net EXTMODE_5V: JP1.7, R9.2, U2.6A
- new net FSYNC: JP6.7, SJ3.2, U7.FSYNC
- new net INT: JP6.8, U7.INT
- new net N$1: C23.1, U7.CPOUT
- new net N$21: C22.1, U7.REGOUT
- new net SCL: JP6.6, R10.1, U7.SCL
- new net SCLK: IC1.SCLK, U2.1Y
- new net SCLK_5V: JP1.4, U2.1A
- new net SCS: IC1.SCS, U2.3Y
- new net SCS_5V: JP1.6, U2.3A
- new net SDA: JP6.5, R11.1, U7.SDA
- new net SI: IC1.SI, U2.2Y
- new net SI_5V: JP1.5, U2.2A
- new net VIN: C20.P$1, JP1.1, U6.EN, U6.IN
- new net VIO: C25.1, JP6.4, U7.VLOGIC
- net GND: now also C17.P$2, C19.P$2, C20.P$2, C21.P$2, C22.2, C23.2, C24.2, C25.2, FB2.P$1, IC1.VSS, JP1.3, JP6.9, R8.2, R9.1, SJ1.3, SJ2.1, SJ3.1, U2.GND, U6.GND, U7.GND
- net VCC: now also C24.1, JP6.10, R10.2, R11.2, SJ1.1, U7.VDD
Other:
- note added: "*"
- note added: "* Two MPU-60X0s can be connected to the same I2C bus"
- note added: "**"
- note added: "** Optional external reference clock input. Connected to GND by default."
- note added: "***"
- note added: "*** Frame synchronization digital input. Connected to GND by default"
- note added: "Added 4 small tcream squares to middle pad."
- note added: "Added selectable jumpers to CLK, FSYNC and AD0"
- note added: "Alternative Address =0x69 (pin AD0 is logic high)"
- note added: "BOM changes"
- note added: "Broke out VLOGIC line"
- note added: "C2 is now 2.2nF instead of 10nF"
- note added: "C2 was mislabled as 10nF, should have been 2.2nF."
- note added: "Changes to V11"
- note added: "Changes to V12: -0402 --> 0603 -Changed Z-Axis symbol to reflect proper orientation from circle with x to circle with dot -Changed NET labels in schematic to flags"
- note added: "Cut trace for external clock"
- note added: "Cut trace for external sync"
- note added: "Default Address = 0x68 (pin AD0 is logic low)"
- note added: "Display On(1)/Off(0)"
- note added: "E. Orosel"
- note added: "FPC: Molex 52892-1095"
- note added: "I2C Address Selection*"
- note added: "J. Bartlett"
- note added: "MOSI"
- note added: "Minor layout changes"
- note added: "New Stencil"
- note added: "Played around with IC footprint."
- note added: "Rounded and elongated pads."
- note added: "SCK"
- note added: "SCL and SDA were switched on V10, fixed on V11"
- note added: "SSEL"
- note added: "The LSB bit of the 7 bit address is determined by the logic level on pin AD0."
- note added: "YES"
- note added: "v12"
