File: EAGLE/project/473/nucleum.brd (EAGLE design)
At the start: 18.8 x 19.6 mm, 40 parts, among them J1 TC2030-JLINK-NL, J2 SH_MALE_2/1MM, J3 ATUM-HEADER, U1 FM25L04B-DG, U3 RV-3049-C3, U4 TPS62740, U5 NRF51822QF, X1 EPSON-FA-128, X2 ABS05-32.768KHZ-T

Commit message: PCB Schematic
Parts:
- added C17: 0.1µF, microbuilder:_0805
- added C18, C19: 1µF, microbuilder:_0805
- added C20, C21: 10µF, microbuilder:_0805
- added C22, C24: 0.1uF, SparkFun:0603-CAP
- added C23: 2.2nF, SparkFun:0603-CAP
- added C25: 10nF, SparkFun:0603-CAP
- added FB1, FB2: (no value), microbuilder:_0805
- added FID1, FID2, FID3: FIDUCIAL"", microbuilder:FIDUCIAL_1MM
- added FRAME4: FRAME-LETTER, SparkFun-Aesthetics:CREATIVE_COMMONS
- added IC1: LS013B4DN04, microbuilder:FPC_10PIN_52892-1095
- added JP1: (no value), microbuilder:1X09_ROUND_70
- added JP2, JP5: FIDUCIALUFIDUCIAL, SparkFun:MICRO-FIDUCIAL
- added JP3, JP4: STAND-OFFTIGHT, SparkFun:STAND-OFF-TIGHT
- added JP6: M10", SparkFun:1X10
- added R10, R11: 10k, SparkFun:0603-RES
- added R7, R8, R9: 10K, microbuilder:_0805
- added SJ1: (no value), SparkFun:SJ_3_PASTE2&3
- added SJ2, SJ3: (no value), SparkFun:SJ_2S-TRACE
- added U$19: (no value), microbuilder:LOGIC_5VREADY_5MM
- added U$21, U$22, U$27, U$28: MOUNTINGHOLE3.0THIN, microbuilder:MOUNTINGHOLE_3.0_PLATEDTHIN
- added U$29: (no value), microbuilder:ADAFRUIT_5MM
- added U$30: OSHW-LOGOS, SparkFun:OSHW-LOGO-S
- added U$31: REVISION, SparkFun-Aesthetics:REVISION
- added U$32, U$33: (no value), SparkFun:SFE-LOGO-FLAME
- added U$34: (no value), SparkFun:SFE-NEW-WEB
- added U2: 74HC4050D, microbuilder:SOIC16
- added U6: MCP1824T-3302E/OT, microbuilder:SOT23-5
- added U7: MPU-6050-1, Testing:QFN-24-4MM2
Connections:
- new net 3.3V: C19.1, C21.1, FB1.1, IC1.P$7, JP1.2, R7.1, U2.1, U6.5
- new net ADO: SJ1.2, U7.9
- new net AGND: C18.2, FB2.2, IC1.P$10
- new net AUX_SCL: JP6.2, U7.7
- new net AUX_SDA: JP6.1, U7.6
- new net AVDD: C18.1, FB1.2, IC1.P$6
- new net CLKIN: JP6.3, SJ2.2, U7.1
- new net DISP: C17.1, IC1.P$5, U2.12
- new net DISP_5V: JP1.8, R7.2, U2.11
- new net EXTCOMIN: IC1.P$4, U2.10
- new net EXTCOMIN_5V: JP1.9, R8.1, U2.9
- new net EXTMODE: IC1.P$8, U2.15
- new net EXTMODE_5V: JP1.7, R9.2, U2.14
- new net FSYNC: JP6.7, SJ3.2, U7.11
- new net INT: JP6.8, U7.12
- new net N$1: C23.1, U7.20
- new net N$21: C22.1, U7.10
- new net SCL: JP6.6, R10.1, U7.23
- new net SCLK: IC1.P$1, U2.2
- new net SCLK_5V: JP1.4, U2.3
- new net SCS: IC1.P$3, U2.6
- new net SCS_5V: JP1.6, U2.7
- new net SDA: JP6.5, R11.1, U7.24
- new net SI: IC1.P$2, U2.4
- new net SI_5V: JP1.5, U2.5
- new net VIN: C20.1, JP1.1, U6.1, U6.3
- new net VIO: C25.1, JP6.4, U7.8
- net GND: now also C17.2, C19.2, C20.2, C21.2, C22.2, C23.2, C24.2, C25.2, FB2.1, IC1.P$9, JP1.3, JP6.9, R8.2, R9.1, SJ1.3, SJ2.1, SJ3.1, U2.8, U6.2, U7.18
- net VCC: now also C24.1, JP6.10, R10.2, R11.2, SJ1.1, U7.13
Routing:
- net 3.3V: track 0.00 -> 55.7 mm, vias 0 -> 3
- net VCC: track 13.8 -> 51.3 mm
- net SI: track 0.00 -> 31.6 mm
- net SCS: track 0.00 -> 31.2 mm
- net SCLK: track 0.00 -> 30.5 mm
- net VIN: track 0.00 -> 27.7 mm
- net EXTCOMIN_5V: track 0.00 -> 27.0 mm, vias 0 -> 1
- net EXTMODE_5V: track 0.00 -> 24.8 mm, vias 0 -> 1
- net DISP_5V: track 0.00 -> 23.8 mm, vias 0 -> 1
- net SCL: track 0.00 -> 20.5 mm, vias 0 -> 1
- net AVDD: track 0.00 -> 19.1 mm
- net SDA: track 0.00 -> 17.3 mm, vias 0 -> 1
- net AUX_SDA: track 0.00 -> 16.2 mm
- net EXTMODE: track 0.00 -> 16.2 mm
- net EXTCOMIN: track 0.00 -> 15.4 mm
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Other:
- board size 18.8 x 19.6 mm -> 40 x 77.2 mm
- board text added: "3V3"
- board text added: "3v3"
- board text added: "AD0"
- board text added: "ASCL"
- board text added: "ASDA"
- board text added: "Adafruit Sharp Memory Disp"
- board text added: "Adafruit!"
- board text added: "CLK"
- board text added: "CS"
- board text added: "DI"
- board text added: "DISP"
- board text added: "Display"
- board text added: "EIN"
- board text added: "EMD"
- board text added: "EXTIN"
- board text added: "EXTMD"
- board text added: "Eric Orosel"
- board text added: "FSYNC"
- board text added: "GND"
- board text added: "INT"
- board text added: "Joel Bartlett"
- board text added: "MOSI"
- board text added: "MPU-6050 Breakout"
- board text added: "Memory"
- board text added: "SCL"
- board text added: "SCLK"
- board text added: "SDA"
- board text added: "SYNC"
- board text added: "Sharp"
- board text added: "V12"
- board text added: "VDD"
- board text added: "VIN"
- board text added: "VIN (3.3-5V)"
- board text added: "VIO"
- board text added: "X"
- board text added: "Y"
- board text added: "Z"
- board text added: "v1.1"
