File: EAGLE/project/FitnessBand/fitnessband.sch (EAGLE design)
At the start: 11 parts, among them U1 RT9193-3.3, U3 FGPMMOPA6H

Commit message: PCB update
Parts:
- removed D2: 1N4148, adafruit:DIODESOD-323F
- removed R6: 10K, rcl:R-US_R0603
- added A1, A2: FRACTUS-2.4GHZ-FR05-S1-N-0-102, chips:FRACTUS-2.4GHZ-FR05-S1-N-0-102
- added B1, B2: BAL-NRF01D3, chips:BAL-NRF01D3
- added BT1, BT2: ML-1220/F1AN, batteries:ML-1220/F1AN
- added C1, C38, C9: 0.1µF, microbuilder:CAP_CERAMIC_0805
- added C10, C11, C3, C39, C40, C6: 1µF, microbuilder:CAP_CERAMIC_0805
- added C12, C16, C18, C20: 0.1uF, SparkFun:CAP0603-CAP
- added C13, C19: 2.2nF, SparkFun:CAP0603-CAP
- added C14, C15, C41, C42, C7, C8: 10µF, microbuilder:CAP_CERAMIC_0805
- added C17, C21: 10nF, SparkFun:CAP0603-CAP
- added C22, C23, C27, C28, C47, C48, C52, C53: 12pF, passives:CAPACITOR
- added C24, C49: 47nF, passives:CAPACITOR
- added C25, C34, C50, C57: 1nF, passives:CAPACITOR
- added C26, C35, C51, C58: 0.1uF, passives:CAPACITOR
- added C29, C54: 10nF, passives:CAPACITOR
- added C30, C31, C61, C62: 10uF, passives:CAPACITOR0603_CAP
- added C32, C55: 2.2nF, passives:CAPACITOR
- added C33, C56: 0.8pF, passives:CAPACITOR
- added C36, C59: 4.7uF, passives:CAPACITOR
- added C37, C60: 1uF, passives:CAPACITOR
- added D1, D3: SML-LX0404SIUPGUSB, leds:SML-LX0404SIUPGUSB
- added FB1, FB2, FB3, FB4, FB5, FB6: (no value), microbuilder:FERRITE_0805
- added FID1, FID2, FID3, FID4, FID5, FID6: FIDUCIAL"", microbuilder:FIDUCIAL""
- added FRAME2: FRAME-LETTER, SparkFun-Aesthetics:FRAME-LETTER
- added IC1, IC2, IC3: LS013B4DN04, microbuilder:SHARP_MEMORYLCD_10PIN
- added J1, J5: TC2030-JLINK-NL, connector:TC2030-JLINK-NL
- added J2, J6: SH_MALE_2/1MM, headers:SH_MALE_2/1MM
- added J3, J4: ATUM-HEADER, atum:ATUM-HEADER
- added JP1, JP2, JP9: (no value), microbuilder:HEADER-1X970MIL
- added JP3, JP4: STAND-OFFTIGHT, SparkFun:STAND-OFFTIGHT
- added JP5, JP6: FIDUCIALUFIDUCIAL, SparkFun:FIDUCIALUFIDUCIAL
- added JP7, JP8: M10", SparkFun:M10"
- added L1, L4: 15nH, passives:INDUCTOR0402
- added L2, L6: 2.2uH, passives:MIPSZ2012D
- added L3, L5: 10uH, passives:INDUCTOR0603
- added LOGO1: UMICH_SOLID_TINY, logos:UMICH_SOLID_TINY
- added R10, R11, R12, R13: 10k, SparkFun:RESISTOR0603-RES
- added R14, R25: 12k, passives:RESISTOR0402_RES
- added R15, R16, R17, R26, R27, R28: 1k, passives:RESISTOR0402_RES
- added R18, R19, R29, R30: 10k, passives:RESISTOR0402_RES
- added R2, R20, R21, R22, R3, R5, R7, R8, R9: 10K, microbuilder:RESISTOR_0805
- added S1, S2: RES_SWITCH, switches:RES_SWITCH
- added SJ1, SJ4: (no value), SparkFun:SOLDERJUMPER_2WAYPASTE2&3
- added SJ2, SJ3, SJ5, SJ6: SOLDERJUMPERTRACE, SparkFun:SOLDERJUMPERTRACE
- added U$21, U$22, U$34, U$35, U$73, U$74, U$86, U$87: MOUNTINGHOLE3.0THIN, microbuilder:MOUNTINGHOLE3.0THIN
- added U$55: OSHW-LOGOS, SparkFun:OSHW-LOGOS
- added U$56: REVISION, SparkFun-Aesthetics:REVISION
- added U10, U19: TPS62740, chips:TPS62740
- added U11, U17: NRF51822QF, chips:NRF51822QF
- added U12, U18: FM25L04B-DG, chips:FM25L04B-DG
- added U13, U2, U5: 74HC4050D, microbuilder:74HC4050D
- added U14, U4, U7: MCP1824T-3302E/OT, microbuilder:VREG_SOT23-5
- added U16, U9: RV-3049-C3, chips:RV-3049-C3
- added U6, U8: MPU-6050-1, Testing:MPU-6050-1
- added X1, X3: EPSON-FA-128, crystals:EPSON-FA-128
- added X2, X4: ABS05-32.768KHZ-T, crystals:ABS05-32.768KHZ-T
Connections:
- removed net RX_5V_GPS: D2.C
- new net !FRAM_CS: U11.P15, U12.!CS, U17.P15, U18.!CS
- new net !FRAM_HOLD: U11.P14, U12.!HOLD, U17.P14, U18.!HOLD
- new net !FRAM_WP: U11.P16, U12.!WP, U17.P16, U18.!WP
- new net !RTC_INT: U11.P25, U16.!INT, U17.P25, U9.!INT
- new net ADO: SJ1.2, SJ4.2, U6.AD0, U8.AD0
- new net AGND: C10.P$2, C3.P$2, C39.P$2, FB2.P$2, FB4.P$2, FB6.P$2, IC1.VSSA, IC2.VSSA, IC3.VSSA
- new net AIN3: J3.25, J4.25, U11.P02/AIN3, U17.P02/AIN3
- new net AIN4: J3.26, J4.26, U11.P03/AIN4, U17.P03/AIN4
- new net AIN5: J3.27, J4.27, U11.P04/AIN5, U17.P04/AIN5
- new net AIN6: J3.28, J4.28, U11.P05/AIN6, U17.P05/AIN6
- new net AIN7: J3.29, J4.29, U11.P06/AIN7/AREF1, U17.P06/AIN7/AREF1
- new net ANTENNA: A1.ANTENNA, B1.SE, C33.1
- new net ANTENNA1: A2.ANTENNA, B2.SE, C56.1
- new net AUX_SCL: JP7.2, JP8.2, U6.AUX_CL, U8.AUX_CL
- new net AUX_SDA: JP7.1, JP8.1, U6.AUX_DA, U8.AUX_DA
- new net AVDD: C10.P$1, C3.P$1, C39.P$1, FB1.P$2, FB3.P$2, FB5.P$2, IC1.VDDA, IC2.VDDA, IC3.VDDA
- new net BATTERY: BT1.+, BT2.+, C30.1, C61.1, J2.2, J3.31, J4.31, J6.2, S1.B, S2.B, U10.EN, U10.VIN, U19.EN, U19.VIN
- new net BOOTLOADER_CTRL: J3.24, J4.24, U11.P13, U17.P13
- new net BOOTLOADER_RX: J3.22, J4.22, U11.P11, U17.P11
- new net BOOTLOADER_TX: J3.23, J4.23, U11.P12, U17.P12
- new net CLKIN: JP7.3, JP8.3, SJ2.2, SJ6.2, U6.CLKIN, U8.CLKIN
- new net DISP: C1.P$1, C38.P$1, C9.P$1, IC1.DISP, IC2.DISP, IC3.DISP, U13.5Y, U2.5Y, U5.5Y
- new net DISP_5V: JP1.8, JP2.8, JP9.8, R2.2, R20.2, R7.2, U13.5A, U2.5A, U5.5A
- new net EXTCOMIN: IC1.EXTCOMIN, IC2.EXTCOMIN, IC3.EXTCOMIN, U13.4Y, U2.4Y, U5.4Y
- new net EXTCOMIN_5V: JP1.9, JP2.9, JP9.9, R21.1, R3.1, R8.1, U13.4A, U2.4A, U5.4A
- new net EXTMODE: IC1.EXTMODE, IC2.EXTMODE, IC3.EXTMODE, U13.6Y, U2.6Y, U5.6Y
- new net EXTMODE_5V: JP1.7, JP2.7, JP9.7, R22.2, R5.2, R9.2, U13.6A, U2.6A, U5.6A
- new net FSYNC: JP7.7, JP8.7, SJ3.2, SJ5.2, U6.FSYNC, U8.FSYNC
- new net I2C_SCL: J3.17, J4.17, U11.P01/AIN2, U17.P01/AIN2
- new net I2C_SDA: J3.18, J4.18, U11.P07, U17.P07
- new net INT: JP7.8, JP8.8, U6.INT, U8.INT
- new net LED_BLUE: R16.1, R27.1, U11.P19, U17.P19
- new net LED_GREEN: R17.1, R28.1, U11.P20, U17.P20
- new net LED_RED: R15.1, R26.1, U11.P18, U17.P18
- new net MOSI_IN: JP1.5, JP2.5, U2.2A, U5.2A
- new net N$10: C23.1, U11.XC2, X1.2
- new net N$11: D1.G, R17.2
- new net N$12: D1.B, R16.2
- new net N$13: C28.1, U11.P27/AIN1/XL1, X2.2
- new net N$14: R19.1, U9.VBACKUP
- new net N$15: C24.1, U11.DEC2
- new net N$16: R18.1, U9.CLKOE
- new net N$17: C25.1, U11.DEC1
- new net N$18: B1.ANT1, U11.ANT1
- new net N$19: B1.ANT2, U11.ANT2
- new net N$20: B1.VDD_PA, C32.1, U11.VDD_PA
- new net N$21: L2.1, U10.SW
- new net N$22: S1.IN, U10.VSEL3, U10.VSEL4
- new net N$25: C47.1, U17.XC1, X3.1
- new net N$26: C48.1, U17.XC2, X3.2
- new net N$27: C49.1, U17.DEC2
- new net N$28: C52.1, U17.P26/AIN0/XL2, X4.1
- new net N$29: C53.1, U17.P27/AIN1/XL1, X4.2
- new net N$3: C13.1, U6.CPOUT
- new net N$30: R30.1, U16.VBACKUP
- new net N$31: R29.1, U16.CLKOE
- new net N$32: C50.1, U17.DEC1
- new net N$33: B2.ANT1, U17.ANT1
- new net N$34: B2.ANT2, U17.ANT2
- new net N$35: B2.VDD_PA, C55.1, U17.VDD_PA
- new net N$36: C34.1, C37.1, L1.1, U11.AVDD
- new net N$37: L1.2, L3.1
- new net N$38: L3.2, U11.DCC
- new net N$39: C57.1, C60.1, L4.1, U17.AVDD
- new net N$4: C19.1, U8.CPOUT
- new net N$40: L4.2, L5.1
- new net N$41: L5.2, U17.DCC
- new net N$42: D3.R, R26.2
- new net N$43: D3.G, R28.2
- new net N$44: D3.B, R27.2
- new net N$45: L6.1, U19.SW
- new net N$46: S2.IN, U19.VSEL3, U19.VSEL4
- new net N$5: C12.1, U6.REGOUT
- new net N$6: C18.1, U8.REGOUT
- new net N$7: C27.1, U11.P26/AIN0/XL2, X2.1
- new net N$8: D1.R, R15.2
- new net N$9: C22.1, U11.XC1, X1.1
- new net P08: J3.19, J4.19, U11.P08, U17.P08
- new net P09: J3.20, J4.20, U11.P09, U17.P09
- new net P10: J3.21, J4.21, U11.P10, U17.P10
- new net P17: J3.2, J4.2, U11.P17, U17.P17
- new net P21: J3.6, J4.6, U11.P21, U17.P21
- new net P22: J3.7, J4.7, U11.P22, U17.P22
- new net P23: J3.8, J4.8, U11.P23, U17.P23
- new net P24: J3.9, J4.9, U11.P24, U17.P24
- new net RTC_CE: U11.P28, U16.CE, U17.P28, U9.CE
- new net SCL: JP7.6, JP8.6, R10.1, R12.1, U6.SCL, U8.SCL
- new net SCLK: IC1.SCLK, IC2.SCLK, IC3.SCLK, U13.1Y, U2.1Y, U5.1Y
- new net SCLK_5V: JP9.4, U13.1A
- new net SCLK_IN: JP1.4, JP2.4, U2.1A, U5.1A
- new net SCS: IC1.SCS, IC2.SCS, IC3.SCS, U13.3Y, U2.3Y, U5.3Y
- new net SCS_5V: JP1.6, JP9.6, U13.3A, U2.3A
- new net SDA: JP7.5, JP8.5, R11.1, R13.1, U6.SDA, U8.SDA
- new net SI: IC1.SI, IC2.SI, IC3.SI, U13.2Y, U2.2Y, U5.2Y
- new net SI_5V: JP9.5, U13.2A
- new net SPI_MISO: J3.14, J4.14, U11.P29, U12.SO, U16.MISO, U17.P29, U18.SO, U9.MISO
- new net SPI_MOSI: J3.15, J4.15, U11.P30, U12.SI, U16.MOSI, U17.P30, U18.SI, U9.MOSI
- new net SPI_SCK: J3.16, J4.16, U11.P00/AREF0, U12.SCK, U16.SCL, U17.P00/AREF0, U18.SCK, U9.SCL
- new net SS_IN: JP2.6, U5.3A
- new net SWDCLK: J1.SWDCLK, J3.4, J4.4, J5.SWDCLK, R14.2, R25.2, U11.SWDCLK, U17.SWDCLK
- new net SWDIO/!RESET: J1.SWDIO, J3.3, J3.30, J4.3, J4.30, J5.SWDIO, U11.SWDIO/!RESET, U17.SWDIO/!RESET
- new net UNUSED1: J3.5, J4.5
- new net UNUSED2: J3.10, J4.10
- new net UNUSED3: J3.11, J4.11
- new net UNUSED4: J3.12, J4.12
- new net UNUSED5: J3.13, J4.13
- new net VCC: C16.1, C20.1, C26.1, C29.1, C31.1, C35.1, C36.1, C51.1, C54.1, C58.1, C59.1, C62.1, D1.VDD, D3.VDD, J1.VCC, J3.1, J4.1, J5.VCC, JP7.10, JP8.10, L2.2, L6.2, R10.2, R11.2, R12.2, R13.2, SJ1.1, SJ4.1, U10.VOUT, U11.VDD, U12.VDD, U16.VCC, U17.VDD, U18.VDD, U19.VOUT, U6.VDD, U8.VDD, U9.VCC
- new net VIO: C17.1, C21.1, JP7.4, JP8.4, U6.VLOGIC, U8.VLOGIC
- net 3.3V: now also C11.P$1, C15.P$1, C40.P$1, C42.P$1, C6.P$1, C8.P$1, FB1.P$1, FB3.P$1, FB5.P$1, IC1.VDD, IC2.VDD, IC3.VDD, JP1.2, JP2.2, JP9.2, R2.1, R20.1, R7.1, U13.VCC, U14.OUT, U2.VCC, U4.OUT, U5.VCC, U7.OUT; no longer R6.2
- net GND: now also B1.GND, B2.GND, BT1.-, BT2.-, C1.P$2, C11.P$2, C12.2, C13.2, C14.P$2, C15.P$2, C16.2, C17.2, C18.2, C19.2, C20.2, C21.2, C22.2, C23.2, C24.2, C25.2, C26.2, C27.2, C28.2, C29.2, C30.2, C31.2, C32.2, C33.2, C34.2, C35.2, C36.2, C37.2, C38.P$2, C40.P$2, C41.P$2, C42.P$2, C47.2, C48.2, C49.2, C50.2, C51.2, C52.2, C53.2, C54.2, C55.2, C56.2, C57.2, C58.2, C59.2, C6.P$2, C60.2, C61.2, C62.2, C7.P$2, C8.P$2, C9.P$2, FB2.P$1, FB4.P$1, FB6.P$1, IC1.VSS, IC2.VSS, IC3.VSS, J1.GND, J2.1, J3.32, J4.32, J5.GND, J6.1, JP1.3, JP2.3, JP7.9, JP8.9, JP9.3, R14.1, R18.2, R19.2, R21.2, R22.1, R25.1, R29.2, R3.2, R30.2, R5.1, R8.2, R9.1, S1.A, S2.A, SJ1.3, SJ2.1, SJ3.1, SJ4.3, SJ5.1, SJ6.1, U10.CTRL, U10.GND, U10.VSEL1, U10.VSEL2, U11.GND, U12.VSS, U13.GND, U14.GND, U16.GND, U17.GND, U18.VSS, U19.CTRL, U19.GND, U19.VSEL1, U19.VSEL2, U2.GND, U4.GND, U5.GND, U6.GND, U7.GND, U8.GND, U9.GND, X1.GND, X3.GND
- net RX_GPS: no longer D2.A, R6.1
- net VIN: now also C14.P$1, C41.P$1, C7.P$1, JP1.1, JP2.1, JP9.1, U14.EN, U14.IN, U4.EN, U4.IN, U7.EN, U7.IN
Other:
- note added: "*"
- note added: "* Two MPU-60X0s can be connected to the same I2C bus"
- note added: "**"
- note added: "** Optional external reference clock input. Connected to GND by default."
- note added: "***"
- note added: "*** Frame synchronization digital input. Connected to GND by default"
- note added: "32 kHz Crystal"
- note added: "4-Kb FRAM"
- note added: "A-1.8V B-3.0V Output"
- note added: "Added 4 small tcream squares to middle pad."
- note added: "Added selectable jumpers to CLK, FSYNC and AD0"
- note added: "Alternative Address =0x69 (pin AD0 is logic high)"
- note added: "BOM changes"
- note added: "Balun"
- note added: "Broke out VLOGIC line"
- note added: "C2 is now 2.2nF instead of 10nF"
- note added: "C2 was mislabled as 10nF, should have been 2.2nF."
- note added: "Changes to V11"
- note added: "Changes to V12: -0402 --> 0603 -Changed Z-Axis symbol to reflect proper orientation from circle with x to circle with dot -Changed NET labels in schematic to flags"
- note added: "Cut trace for external clock"
- note added: "Cut trace for external sync"
- note added: "Default Address = 0x68 (pin AD0 is logic low)"
- note added: "Display On(1)/Off(0)"
- note added: "E. Orosel"
- note added: "FPC: Molex 52892-1095"
- note added: "GPS"
- note added: "I2C Address Selection*"
- note added: "IMU"
- note added: "J-Link"
- note added: "J. Bartlett"
- note added: "LCD"
- note added: "MOSI"
- note added: "Mhz Range Crystal"
- note added: "Minor layout changes"
- note added: "New Stencil"
- note added: "Played around with IC footprint."
- note added: "Real Time Clock"
- note added: "Rounded and elongated pads."
- note added: "SCK"
- note added: "SCL and SDA were switched on V10, fixed on V11"
- note added: "SSEL"
- note added: "Sup"
- note added: "The LSB bit of the 7 bit address is determined by the logic level on pin AD0."
- note added: "YES"
- note added: "nucleum"
- note added: "nucleum power"
- note added: "v12"

Commit message: I'm tired so I'm not writing a good commit message
Parts:
- removed BT2: ML-1220/F1AN, batteries:ML-1220/F1AN
- removed L6: 2.2uH, passives:MIPSZ2012D
- removed S2: RES_SWITCH, switches:RES_SWITCH
- removed SJ4: (no value), SparkFun:SOLDERJUMPER_2WAYPASTE2&3
- removed SJ5, SJ6: SOLDERJUMPERTRACE, SparkFun:SOLDERJUMPERTRACE
- removed U19: TPS62740, chips:TPS62740
- added C43, C44: 1uF, resistor:C-EUC0603
- added C45: (no value), resistor:C-EUC0603
- added C46: 1uF, SparkFun:CAP0402-CAP
- added C63: 10nF, SparkFun:CAP0402-CAP
- added IC4: MAX1555, maxim:MAX1555
- added IC5: LP2951M, national-semiconductor:LP2951M
- added JP10: (no value), SparkFun:M03PTH
- added JP11: LOGO-SFESK, SparkFun:LOGO-SFESK
- added JP12: (no value), SparkFun:M02PTH
- added JP13, JP14: FIDUCIAL1X2.5, abes:FIDUCIAL1X2.5
- added R23: 180, SparkFun:RESISTOR0402-RES
- added R24, R31, R32, R33, R34, R35, R36, R37: 4.7k, SparkFun:RESISTOR0402-RES
- added R6: 100k, resistor:R-US_R0603
- added U$59: OSHW-LOGOS, SparkFun:OSHW-LOGOS
- added U15: MAX1704X, SparkFun:MAX1704X
- C61: value 10uF -> 10nF; device passives:CAPACITOR0603_CAP -> SparkFun:CAP0402-CAP; DIGIKEY 490-7316-1-ND -> (none)
- C62: value 10uF -> 1uF; device passives:CAPACITOR0603_CAP -> SparkFun:CAP0402-CAP; DIGIKEY 490-7316-1-ND -> (none)
- JP2: value (none) -> input; device microbuilder:HEADER-1X970MIL -> SparkFun:M02-JST-2MM-SMT
- JP8: value M10" -> (none); device SparkFun:M10" -> SparkFun:M03PTH
- R7, R9: value 10K -> 1k; device microbuilder:RESISTOR_0805 -> SparkFun:RESISTOR0402-RES
- R8: value 10K -> 180; device microbuilder:RESISTOR_0805 -> SparkFun:RESISTOR0402-RES
- U5: value 74HC4050D -> MAX1704X; device microbuilder:74HC4050D -> SparkFun:MAX1704X
Connections:
- removed net SS_IN: JP2.6, U5.3A
- new net AGLCD: C10.P$2, FB4.P$2, IC2.VSSA
- new net ALCD: C10.P$1, FB3.P$2, IC2.VDDA
- new net ALT: JP10.3, R24.1, U5.ALT
- new net ALT_FG: R34.1, U15.ALT
- new net CHARGING?: IC4.!CHG, R6.1
- new net IMU_INT: U8.INT
- new net N$47: C62.1, R7.2, U15.CELL
- new net QST: JP8.3, R31.2, U5.QST
- new net QST_FG: R35.2, U15.QST
- new net SCL_FG: R36.1, U15.SCL
- new net SDA_FG: R37.1, U15.SDA
- new net USB_PORT: C44.1, IC4.USB
- new net VDD: C61.1, C63.1, R23.1, R8.1, U15.VDD, U5.VDD
- net 3.3V: now also C20.1, C21.1, C45.2, C9.P$1, IC2.DISP, IC5.OUT, IC5.SENSE, R12.2, R13.2, R34.2, R36.2, R37.2, R6.2, U8.VDD, U8.VLOGIC; no longer JP2.2, R7.1, U5.VCC
- net ADO: no longer SJ4.2, U8.AD0
- net AGND: no longer C10.P$2, FB4.P$2, IC2.VSSA
- net AUX_SCL: no longer JP8.2, U8.AUX_CL
- net AUX_SDA: no longer JP8.1, U8.AUX_DA
- net AVDD: no longer C10.P$1, FB3.P$2, IC2.VDDA
- net BATTERY: now also C43.1, IC4.BAT, IC5.VIN, R7.1, R8.2; no longer BT2.+, C61.1, S2.B, U19.EN, U19.VIN
- net CLKIN: no longer JP8.3, SJ6.2, U8.CLKIN
- net DISP: no longer C9.P$1, IC2.DISP, U5.5Y
- net DISP_5V: no longer JP2.8, R7.2, U5.5A
- net EXTCOMIN: no longer IC2.EXTCOMIN, U5.4Y
- net EXTCOMIN_5V: no longer JP2.9, R8.1, U5.4A
- net EXTMODE: no longer IC2.EXTMODE, U5.6Y
- net EXTMODE_5V: no longer JP2.7, R9.2, U5.6A
- net FSYNC: no longer JP8.7, SJ5.2, U8.FSYNC
- net GND: now also C43.2, C44.2, C45.1, C46.2, C63.2, IC2.EXTCOMIN, IC2.EXTMODE, IC4.GND, IC5.GND, IC5.SHDWN, JP10.2, JP12.2, JP2.1, R31.1, R35.1, U15.CTG, U15.GND@4, U15.GND@EP, U5.CTG, U5.GND@4, U5.GND@EP, U8.AD0, U8.CLKIN, U8.FSYNC; no longer BT2.-, JP2.3, JP8.9, R8.2, R9.1, S2.A, SJ4.3, SJ5.1, SJ6.1, U19.CTRL, U19.GND, U19.VSEL1, U19.VSEL2, U5.GND
- net INT: no longer JP8.8, U8.INT
- net MOSI_IN: no longer JP2.5, U5.2A
- net N$45: now also C46.1, R9.2, U5.CELL; no longer L6.1, U19.SW
- net N$46: now also IC5.FB, IC5.VTAB; no longer S2.IN, U19.VSEL3, U19.VSEL4
- net SCL: now also JP8.2, R32.1, U5.SCL; no longer JP8.6
- net SCLK: no longer U5.1Y
- net SCLK_IN: no longer JP2.4, U5.1A
- net SCS: no longer U5.3Y
- net SDA: now also JP8.1, R33.1, U5.SDA; no longer JP8.5
- net SI: no longer U5.2Y
- net VCC: now also JP10.1, JP12.1, JP2.2, R23.2, R24.2, R32.2, R33.2, R9.1; no longer C20.1, C62.1, JP8.10, L6.2, R12.2, R13.2, SJ4.1, U19.VOUT, U8.VDD
- net VIN: no longer JP2.1
- net VIO: no longer C21.1, JP8.4, U8.VLOGIC
Other:
- note added: "BATTERY"
- note added: "CHARGER"
- note added: "Do we want this connector or pads?"
- note added: "Fuel Gauge"
- note added: "LDO"
- note added: "NEEDS A VAl!"
- note removed: "D1+R3 restrict RX input to 3.3V"

Commit message: asdf
Parts:
- removed C51: 0.1uF, passives:CAPACITOR
- removed C54: 10nF, passives:CAPACITOR
- removed J4: ATUM-HEADER, atum:ATUM-HEADER
- removed R29, R30: 10k, passives:RESISTOR0402_RES
- removed U16: RV-3049-C3, chips:RV-3049-C3
- removed U18: FM25L04B-DG, chips:FM25L04B-DG
Connections:
- removed net N$30: R30.1, U16.VBACKUP
- removed net N$31: R29.1, U16.CLKOE
- new net SCLK_LCD: IC2.SCLK
- new net SCS_LCD: IC2.SCS
- new net SI_LCD: IC2.SI
- net !FRAM_CS: no longer U18.!CS
- net !FRAM_HOLD: no longer U18.!HOLD
- net !FRAM_WP: no longer U18.!WP
- net !RTC_INT: no longer U16.!INT
- net AIN3: no longer J4.25
- net AIN4: no longer J4.26
- net AIN5: no longer J4.27
- net AIN6: no longer J4.28
- net AIN7: no longer J4.29
- net BATTERY: no longer J4.31
- net BOOTLOADER_CTRL: no longer J4.24
- net BOOTLOADER_RX: no longer J4.22
- net BOOTLOADER_TX: no longer J4.23
- net GND: no longer C51.2, C54.2, J4.32, R29.2, R30.2, U16.GND, U18.VSS
- net I2C_SCL: no longer J4.17
- net I2C_SDA: no longer J4.18
- net P08: no longer J4.19, U17.P08
- net P09: no longer J4.20, U17.P09
- net P10: no longer J4.21
- net P17: no longer J4.2
- net P21: no longer J4.6
- net P22: no longer J4.7
- net P23: no longer J4.8
- net P24: no longer J4.9
- net RTC_CE: no longer U16.CE
- net RX_GPS: now also U17.P09
- net SCLK: no longer IC2.SCLK
- net SCS: no longer IC2.SCS
- net SI: no longer IC2.SI
- net SPI_MISO: no longer J4.14, U16.MISO, U18.SO
- net SPI_MOSI: no longer J4.15, U16.MOSI, U18.SI
- net SPI_SCK: no longer J4.16, U16.SCL, U18.SCK
- net SWDCLK: no longer J4.4
- net SWDIO/!RESET: no longer J4.3, J4.30
- net TX_GPS: now also U17.P08
- net UNUSED1: no longer J4.5
- net UNUSED2: no longer J4.10
- net UNUSED3: no longer J4.11
- net UNUSED4: no longer J4.12
- net UNUSED5: no longer J4.13
- net VCC: no longer C51.1, C54.1, J4.1, U16.VCC, U18.VDD
Other:
- note added: "NEED A MICRO USB PORT"
- note removed: "4-Kb FRAM"
- note removed: "Real Time Clock"
- moved on the sheet: J5

Commit message: combined sheets
Parts:
- removed C18, C20: 0.1uF, SparkFun:CAP0603-CAP
- removed C19: 2.2nF, SparkFun:CAP0603-CAP
- removed C2: 0.1uF, resistor:C-EUC0603
- removed C21: 10nF, SparkFun:CAP0603-CAP
- removed LED2: FIX, microbuilder:LED0805
- removed R12, R13: 10k, SparkFun:RESISTOR0603-RES
- removed R4: 1K, rcl:R-US_R0603
- removed U3: FGPMMOPA6H, microbuilder:GPS_FGPMMOPA6H
- removed U8: MPU-6050-1, Testing:MPU-6050-1
- added C51: 0.1uF, resistor:C-EUC0603
- added C54, C65: 0.1uF, SparkFun:CAP0603-CAP
- added C64: 2.2nF, SparkFun:CAP0603-CAP
- added C66: 10nF, SparkFun:CAP0603-CAP
- added LED1: FIX, microbuilder:LED0805
- added R29: 1K, rcl:R-US_R0603
- added R30, R38: 10k, SparkFun:RESISTOR0603-RES
- added U16: FGPMMOPA6H, microbuilder:GPS_FGPMMOPA6H
- added U18: MPU-6050-1, Testing:MPU-6050-1
Connections:
- removed net N$1: LED2.C, R4.2
- removed net N$4: C19.1, U8.CPOUT
- removed net N$6: C18.1, U8.REGOUT
- new net N$23: LED1.C, R29.2
- new net N$48: C64.1, U18.CPOUT
- new net N$49: C54.1, U18.REGOUT
- net 1PPS: now also U16.1PPS; no longer U3.1PPS
- net 3.3V: now also C51.1, C65.1, C66.1, R30.2, R38.2, U16.VCC, U18.VDD, U18.VLOGIC; no longer C2.1, C20.1, C21.1, R12.2, R13.2, U3.VCC, U8.VDD, U8.VLOGIC
- net FIX: now also LED1.A, U16.3D-FIX; no longer LED2.A, U3.3D-FIX
- net GND: now also C51.2, C54.2, C64.2, C65.2, C66.2, R29.1, U16.GND@1, U16.GND@2, U16.GND@3, U16.GND@4, U18.AD0, U18.CLKIN, U18.FSYNC, U18.GND; no longer C18.2, C19.2, C2.2, C20.2, C21.2, R4.1, U3.GND@1, U3.GND@2, U3.GND@3, U3.GND@4, U8.AD0, U8.CLKIN, U8.FSYNC, U8.GND
- net IMU_INT: now also U18.INT; no longer U8.INT
- net RX_GPS: now also U16.RX; no longer U3.RX
- net SCL: now also R30.1, U18.SCL; no longer R12.1, U8.SCL
- net SDA: now also R38.1, U18.SDA; no longer R13.1, U8.SDA
- net TX_GPS: now also U16.TX; no longer U3.TX

Commit message: wow
Parts:
- removed A1: FRACTUS-2.4GHZ-FR05-S1-N-0-102, chips:FRACTUS-2.4GHZ-FR05-S1-N-0-102
- removed B1: BAL-NRF01D3, chips:BAL-NRF01D3
- removed BT1: ML-1220/F1AN, batteries:ML-1220/F1AN
- removed C1, C38, C9: 0.1µF, microbuilder:CAP_CERAMIC_0805
- removed C10, C11, C39, C40, C6: 1µF, microbuilder:CAP_CERAMIC_0805
- removed C12, C16, C54, C65: 0.1uF, SparkFun:CAP0603-CAP
- removed C13, C64: 2.2nF, SparkFun:CAP0603-CAP
- removed C14, C15, C41, C42, C7, C8: 10µF, microbuilder:CAP_CERAMIC_0805
- removed C17, C66: 10nF, SparkFun:CAP0603-CAP
- removed C22, C23, C27, C28: 12pF, passives:CAPACITOR
- removed C24: 47nF, passives:CAPACITOR
- removed C25, C34: 1nF, passives:CAPACITOR
- removed C26, C35: 0.1uF, passives:CAPACITOR
- removed C29: 10nF, passives:CAPACITOR
- removed C30, C31: 10uF, passives:CAPACITOR0603_CAP
- removed C32: 2.2nF, passives:CAPACITOR
- removed C33: 0.8pF, passives:CAPACITOR
- removed C36: 4.7uF, passives:CAPACITOR
- removed C37, C60: 1uF, passives:CAPACITOR
- removed C43, C44: 1uF, resistor:C-EUC0603
- removed C45: (no value), resistor:C-EUC0603
- removed C46: 1uF, SparkFun:CAP0402-CAP
- removed C51: 0.1uF, resistor:C-EUC0603
- removed C61: 10nF, SparkFun:CAP0402-CAP
- removed D1, D3: SML-LX0404SIUPGUSB, leds:SML-LX0404SIUPGUSB
- removed FB1, FB2, FB5, FB6: (no value), microbuilder:FERRITE_0805
- removed FERRITE2: INDUCTOR, resistor:C-EUC0805
- removed FID1, FID2, FID3, FID4, FID5, FID6: FIDUCIAL"", microbuilder:FIDUCIAL""
- removed FRAME2: FRAME-LETTER, SparkFun-Aesthetics:FRAME-LETTER
- removed IC1, IC3: LS013B4DN04, microbuilder:SHARP_MEMORYLCD_10PIN
- removed J1: TC2030-JLINK-NL, connector:TC2030-JLINK-NL
- removed J2: SH_MALE_2/1MM, headers:SH_MALE_2/1MM
- removed J3: ATUM-HEADER, atum:ATUM-HEADER
- removed JP1, JP9: (no value), microbuilder:HEADER-1X970MIL
- removed JP10, JP8: (no value), SparkFun:M03PTH
- removed JP11: LOGO-SFESK, SparkFun:LOGO-SFESK
- removed JP12: (no value), SparkFun:M02PTH
- removed JP13, JP14: FIDUCIAL1X2.5, abes:FIDUCIAL1X2.5
- removed JP2: input, SparkFun:M02-JST-2MM-SMT
- removed JP3, JP4: STAND-OFFTIGHT, SparkFun:STAND-OFFTIGHT
- removed JP5, JP6: FIDUCIALUFIDUCIAL, SparkFun:FIDUCIALUFIDUCIAL
- removed JP7: M10", SparkFun:M10"
- removed L1, L4: 15nH, passives:INDUCTOR0402
- removed L2: 2.2uH, passives:MIPSZ2012D
- removed L3, L5: 10uH, passives:INDUCTOR0603
- removed LOGO1: UMICH_SOLID_TINY, logos:UMICH_SOLID_TINY
- removed R11, R30, R38: 10k, SparkFun:RESISTOR0603-RES
- removed R14: 12k, passives:RESISTOR0402_RES
- removed R15, R16, R17, R26, R27, R28: 1k, passives:RESISTOR0402_RES
- removed R18, R19: 10k, passives:RESISTOR0402_RES
- removed R20, R21, R22, R5: 10K, microbuilder:RESISTOR_0805
- removed R23: 180, SparkFun:RESISTOR0402-RES
- removed R24, R31, R32, R33: 4.7k, SparkFun:RESISTOR0402-RES
- removed R29: 1K, rcl:R-US_R0603
- removed R6: 100k, resistor:R-US_R0603
- removed R9: 1k, SparkFun:RESISTOR0402-RES
- removed S1: RES_SWITCH, switches:RES_SWITCH
- removed SJ1: (no value), SparkFun:SOLDERJUMPER_2WAYPASTE2&3
- removed SJ2, SJ3: SOLDERJUMPERTRACE, SparkFun:SOLDERJUMPERTRACE
- removed U$21, U$22, U$34, U$35, U$73, U$74, U$86, U$87: MOUNTINGHOLE3.0THIN, microbuilder:MOUNTINGHOLE3.0THIN
- removed U$55, U$59: OSHW-LOGOS, SparkFun:OSHW-LOGOS
- removed U$56: REVISION, SparkFun-Aesthetics:REVISION
- removed U1: RT9193-3.3, microbuilder:VREG_SOT23-5
- removed U10: TPS62740, chips:TPS62740
- removed U11: NRF51822QF, chips:NRF51822QF
- removed U12: FM25L04B-DG, chips:FM25L04B-DG
- removed U13, U2: 74HC4050D, microbuilder:74HC4050D
- removed U14, U4, U7: MCP1824T-3302E/OT, microbuilder:VREG_SOT23-5
- removed U5: MAX1704X, SparkFun:MAX1704X
- removed U6: MPU-6050-1, Testing:MPU-6050-1
- removed U9: RV-3049-C3, chips:RV-3049-C3
- removed X1: EPSON-FA-128, crystals:EPSON-FA-128
- removed X2: ABS05-32.768KHZ-T, crystals:ABS05-32.768KHZ-T
- added C12_IMU, C13_IMU, C16_LCD, C_FRAM: 0.1uF, resistor:C-EUC0402
- added C14_LCD, C15_LCD, C2: 1uF, resistor:C-EUC0402
- added C7_IMU: 10nF, resistor:C-EUC0402
- added C8_IMU: 2.2uF, resistor:C-EUC0402
- added FRAM: FM25L04B-DG, chips:FM25L04B-DG
- added JP16: M11LOCK, SparkFun:M11LOCK
- added R4: 1K, resistor:R-US_R0402
- added R5_IMU, R9_IMU: 10K, resistor:R-US_R0402
- added RGB_LED: SML-LX0404SIUPGUSB, leds:SML-LX0404SIUPGUSB
- added X5: USB-MICROB, SparkFun:USB-MICROB
- C3: value 1µF -> 1uF; device microbuilder:CAP_CERAMIC_0805 -> resistor:C-EUC0402
- C4: value 10uF -> (none); device resistor:C-EUC0603 -> resistor:C-EUC0402
- C5: value 10uF -> 0.1uF; device resistor:C-EUC0603 -> resistor:C-EUC0402
- C58: value 0.1uF -> 100nF
- C59: value 4.7uF -> 100nF
- R1: value 10K -> 1k; device rcl:R-US_R0603 -> passives:RESISTOR0402_RES
- R10: value 10k -> 100K; device SparkFun:RESISTOR0603-RES -> resistor:R-US_R0402
- R2, R3: value 10K -> 1k; device microbuilder:RESISTOR_0805 -> passives:RESISTOR0402_RES
- renumbered A2 to ANT, B2 to BALUN, IC2 to LCD_PORT, IC4 to CHARGER, IC5 to LDO, J6 to B_CONNECTOR, U15 to FG, U16 to GPS, U18 to IMU
Connections:
- removed net !RTC_INT: U11.P25, U17.P25, U9.!INT
- removed net 1PPS: GPS.1PPS
- removed net ADO: SJ1.2, U6.AD0
- removed net AGND: C3.P$2, C39.P$2, FB2.P$2, FB6.P$2, IC1.VSSA, IC3.VSSA
- removed net AIN3: J3.25, U11.P02/AIN3, U17.P02/AIN3
- removed net AIN4: J3.26, U11.P03/AIN4, U17.P03/AIN4
- removed net AIN5: J3.27, U11.P04/AIN5, U17.P04/AIN5
- removed net AIN6: J3.28, U11.P05/AIN6, U17.P05/AIN6
- removed net AIN7: J3.29, U11.P06/AIN7/AREF1, U17.P06/AIN7/AREF1
- removed net ALT: JP10.3, R24.1, U5.ALT
- removed net ANTENNA: A1.ANTENNA, B1.SE, C33.1
- removed net AUX_SCL: JP7.2, U6.AUX_CL
- removed net AUX_SDA: JP7.1, U6.AUX_DA
- removed net AVDD: C3.P$1, C39.P$1, FB1.P$2, FB5.P$2, IC1.VDDA, IC3.VDDA
- removed net BOOTLOADER_CTRL: J3.24, U11.P13, U17.P13
- removed net BOOTLOADER_RX: J3.22, U11.P11, U17.P11
- removed net BOOTLOADER_TX: J3.23, U11.P12, U17.P12
- removed net CLKIN: JP7.3, SJ2.2, U6.CLKIN
- removed net DISP: C1.P$1, C38.P$1, IC1.DISP, IC3.DISP, U13.5Y, U2.5Y
- removed net DISP_5V: JP1.8, JP9.8, R2.2, R20.2, U13.5A, U2.5A
- removed net ENABLE: R1.1, U1.EN
- removed net EXTCOMIN: IC1.EXTCOMIN, IC3.EXTCOMIN, U13.4Y, U2.4Y
- removed net EXTCOMIN_5V: JP1.9, JP9.9, R21.1, R3.1, U13.4A, U2.4A
- removed net EXTMODE: IC1.EXTMODE, IC3.EXTMODE, U13.6Y, U2.6Y
- removed net EXTMODE_5V: JP1.7, JP9.7, R22.2, R5.2, U13.6A, U2.6A
- removed net FSYNC: JP7.7, SJ3.2, U6.FSYNC
- removed net I2C_SCL: J3.17, U11.P01/AIN2, U17.P01/AIN2
- removed net I2C_SDA: J3.18, U11.P07, U17.P07
- removed net IMU_INT: IMU.INT
- removed net INT: JP7.8, U6.INT
- removed net MOSI_IN: JP1.5, U2.2A
- removed net N$10: C23.1, U11.XC2, X1.2
- removed net N$11: D1.G, R17.2
- removed net N$12: D1.B, R16.2
- removed net N$13: C28.1, U11.P27/AIN1/XL1, X2.2
- removed net N$14: R19.1, U9.VBACKUP
- removed net N$15: C24.1, U11.DEC2
- removed net N$16: R18.1, U9.CLKOE
- removed net N$17: C25.1, U11.DEC1
- removed net N$18: B1.ANT1, U11.ANT1
- removed net N$19: B1.ANT2, U11.ANT2
- removed net N$20: B1.VDD_PA, C32.1, U11.VDD_PA
- removed net N$21: L2.1, U10.SW
- removed net N$22: S1.IN, U10.VSEL3, U10.VSEL4
- removed net N$36: C34.1, C37.1, L1.1, U11.AVDD
- removed net N$37: L1.2, L3.1
- removed net N$38: L3.2, U11.DCC
- removed net N$39: C57.1, C60.1, L4.1, U17.AVDD
- removed net N$40: L4.2, L5.1
- removed net N$41: L5.2, U17.DCC
- removed net N$42: D3.R, R26.2
- removed net N$43: D3.G, R28.2
- removed net N$44: D3.B, R27.2
- removed net N$45: C46.1, R9.2, U5.CELL
- removed net N$5: C12.1, U6.REGOUT
- removed net N$7: C27.1, U11.P26/AIN0/XL2, X2.1
- removed net N$8: D1.R, R15.2
- removed net N$9: C22.1, U11.XC1, X1.1
- removed net P08: J3.19, U11.P08
- removed net P09: J3.20, U11.P09
- removed net P10: J3.21, U11.P10, U17.P10
- removed net P17: J3.2, U11.P17, U17.P17
- removed net P21: J3.6, U11.P21, U17.P21
- removed net P22: J3.7, U11.P22, U17.P22
- removed net P23: J3.8, U11.P23, U17.P23
- removed net P24: J3.9, U11.P24, U17.P24
- removed net QST: JP8.3, R31.2, U5.QST
- removed net RTC_CE: U11.P28, U17.P28, U9.CE
- removed net SCL: IMU.SCL, JP7.6, JP8.2, R10.1, R30.1, R32.1, U5.SCL, U6.SCL
- removed net SCLK: IC1.SCLK, IC3.SCLK, U13.1Y, U2.1Y
- removed net SCLK_5V: JP9.4, U13.1A
- removed net SCLK_IN: JP1.4, U2.1A
- removed net SCS: IC1.SCS, IC3.SCS, U13.3Y, U2.3Y
- removed net SCS_5V: JP1.6, JP9.6, U13.3A, U2.3A
- removed net SDA: IMU.SDA, JP7.5, JP8.1, R11.1, R33.1, R38.1, U5.SDA, U6.SDA
- removed net SI: IC1.SI, IC3.SI, U13.2Y, U2.2Y
- removed net SI_5V: JP9.5, U13.2A
- removed net SPI_MISO: J3.14, U11.P29, U12.SO, U17.P29, U9.MISO
- removed net SPI_MOSI: J3.15, U11.P30, U12.SI, U17.P30, U9.MOSI
- removed net SPI_SCK: J3.16, U11.P00/AREF0, U12.SCK, U17.P00/AREF0, U9.SCL
- removed net UNUSED1: J3.5
- removed net UNUSED2: J3.10
- removed net UNUSED3: J3.11
- removed net UNUSED4: J3.12
- removed net UNUSED5: J3.13
- removed net VCC: C16.1, C26.1, C29.1, C31.1, C35.1, C36.1, C58.1, C59.1, D1.VDD, D3.VDD, J1.VCC, J3.1, J5.VCC, JP10.1, JP12.1, JP2.2, JP7.10, L2.2, R10.2, R11.2, R23.2, R24.2, R32.2, R33.2, R9.1, SJ1.1, U10.VOUT, U11.VDD, U12.VDD, U17.VDD, U6.VDD, U9.VCC
- removed net VIN: C14.P$1, C4.1, C41.P$1, C7.P$1, JP1.1, JP9.1, R1.2, U1.IN, U14.EN, U14.IN, U4.EN, U4.IN, U7.EN, U7.IN
- removed net VIO: C17.1, JP7.4, U6.VLOGIC
- new net BUTTON1: JP16.11, U17.P21
- new net BUTTON2: JP16.7, U17.P22
- new net BUTTON3: JP16.3, U17.P23
- new net GPIO1: JP16.8, U17.P17
- new net HR: JP16.10, U17.P01/AIN2
- new net INT_IMU: IMU.INT, U17.P28
- new net N$1: R1.2, RGB_LED.R
- new net SCL_IMU: IMU.SCL, R5_IMU.1, U17.P24
- new net SDA_IMU: IMU.SDA, R9_IMU.1, U17.P25
- new net SPI_MISO_FRAM: FRAM.SO, U17.P29
- new net SPI_MOSI_FRAM: FRAM.SI, U17.P30
- new net SPI_SCK_FRAM: FRAM.SCK, U17.P00/AREF0
- net !FRAM_CS: now also FRAM.!CS; no longer U11.P15, U12.!CS
- net !FRAM_HOLD: now also FRAM.!HOLD; no longer U11.P14, U12.!HOLD
- net !FRAM_WP: now also FRAM.!WP; no longer U11.P16, U12.!WP
- net 3.3V: now also C13_IMU.1, C14_LCD.1, C16_LCD.1, C4.1, C57.1, C58.1, C59.1, C7_IMU.1, C_FRAM.1, FRAM.VDD, J5.VCC, JP16.4, R10.2, R5_IMU.2, R9_IMU.2, RGB_LED.VDD, U17.AVDD, U17.VDD; no longer C11.P$1, C15.P$1, C40.P$1, C42.P$1, C45.2, C51.1, C6.P$1, C65.1, C66.1, C8.P$1, C9.P$1, FB1.P$1, FB5.P$1, FERRITE2.2, IC1.VDD, IC3.VDD, JP1.2, JP9.2, R2.1, R20.1, R30.2, R38.2, R6.2, U13.VCC, U14.OUT, U2.VCC, U4.OUT, U7.OUT
- net AGLCD: now also C15_LCD.2; no longer C10.P$2
- net ALCD: now also C15_LCD.1; no longer C10.P$1
- net ALT_FG: now also U17.P13
- net BATTERY: now also C3.1; no longer BT1.+, C30.1, C43.1, J2.2, J3.31, S1.B, U10.EN, U10.VIN
- net CHARGING?: now also R10.1; no longer R6.1
- net GND: now also C12_IMU.2, C13_IMU.2, C14_LCD.2, C16_LCD.2, C2.2, C3.2, C7_IMU.2, C8_IMU.2, C_FRAM.2, FRAM.VSS, JP16.1, JP16.5, JP16.9, R4.1, X5.GND; no longer B1.GND, BT1.-, C1.P$2, C11.P$2, C12.2, C13.2, C14.P$2, C15.P$2, C16.2, C17.2, C22.2, C23.2, C24.2, C25.2, C26.2, C27.2, C28.2, C29.2, C30.2, C31.2, C32.2, C33.2, C34.2, C35.2, C36.2, C37.2, C38.P$2, C40.P$2, C41.P$2, C42.P$2, C43.2, C44.2, C45.1, C46.2, C51.2, C54.2, C6.P$2, C60.2, C61.2, C64.2, C65.2, C66.2, C7.P$2, C8.P$2, C9.P$2, FB2.P$1, FB6.P$1, IC1.VSS, IC3.VSS, J1.GND, J2.1, J3.32, JP1.3, JP10.2, JP12.2, JP2.1, JP7.9, JP9.3, R14.1, R18.2, R19.2, R21.2, R22.1, R29.1, R3.2, R31.1, R5.1, S1.A, SJ1.3, SJ2.1, SJ3.1, U1.GND, U10.CTRL, U10.GND, U10.VSEL1, U10.VSEL2, U11.GND, U12.VSS, U13.GND, U14.GND, U2.GND, U4.GND, U5.CTG, U5.GND@4, U5.GND@EP, U6.GND, U7.GND, U9.GND, X1.GND
- net LED_BLUE: now also R2.1; no longer R16.1, R27.1, U11.P19
- net LED_GREEN: now also R3.1; no longer R17.1, R28.1, U11.P20
- net LED_RED: now also R1.1; no longer R15.1, R26.1, U11.P18
- net N$2: now also R3.2, RGB_LED.G; no longer FERRITE2.1, U1.OUT
- net N$23: now also R4.2; no longer R29.2
- net N$3: now also R2.2, RGB_LED.B; no longer C13.1, U6.CPOUT
- net N$48: now also C8_IMU.1; no longer C64.1
- net N$49: now also C12_IMU.1; no longer C54.1
- net QST_FG: now also U17.P12
- net SCLK_LCD: now also U17.P05/AIN6
- net SCL_FG: now also U17.P11
- net SCS_LCD: now also U17.P07
- net SDA_FG: now also U17.P10
- net SI_LCD: now also U17.P06/AIN7/AREF1
- net SWDCLK: no longer J1.SWDCLK, J3.4, R14.2, U11.SWDCLK
- net SWDIO/!RESET: no longer J1.SWDIO, J3.3, J3.30, U11.SWDIO/!RESET
- net USB_PORT: now also C2.1, X5.VBUS; no longer C44.1
- net VDD: no longer C61.1, R23.1, U5.VDD
Other:
- note removed: "* Two MPU-60X0s can be connected to the same I2C bus"
- note removed: "**"
- note removed: "** Optional external reference clock input. Connected to GND by default."
- note removed: "***"
- note removed: "*** Frame synchronization digital input. Connected to GND by default"
- note removed: "A-1.8V B-3.0V Output"
- note removed: "Added 4 small tcream squares to middle pad."
- note removed: "Added selectable jumpers to CLK, FSYNC and AD0"
- note removed: "Alternative Address =0x69 (pin AD0 is logic high)"
- note removed: "BOM changes"
- note removed: "Broke out VLOGIC line"
- note removed: "C2 is now 2.2nF instead of 10nF"
- note removed: "C2 was mislabled as 10nF, should have been 2.2nF."
- note removed: "Changes to V11"
- note removed: "Changes to V12: -0402 --> 0603 -Changed Z-Axis symbol to reflect proper orientation from circle with x to circle with dot -Changed NET labels in schematic to flags"
- note removed: "Cut trace for external clock"
- note removed: "Cut trace for external sync"
- note removed: "Default Address = 0x68 (pin AD0 is logic low)"
- note removed: "Display On(1)/Off(0)"
- note removed: "E. Orosel"
- note removed: "J. Bartlett"
- note removed: "MOSI"
- note removed: "Minor layout changes"
- note removed: "NEED A MICRO USB PORT"
- note removed: "New Stencil"
- note removed: "Played around with IC footprint."
- note removed: "Rounded and elongated pads."
- note removed: "SCK"
- note removed: "SCL and SDA were switched on V10, fixed on V11"
- note removed: "SSEL"
- note removed: "Sup"
- note removed: "The LSB bit of the 7 bit address is determined by the logic level on pin AD0."
- note removed: "YES"
- note removed: "nucleum"
- note removed: "nucleum power"
- note removed: "v12"

Commit message: began layot
Parts:
- renumbered C2 to C2_CH, C3 to C3_CH, C4 to C4_LDO, C5 to C5_GPS, C62 to C62_FG, C63 to C63_FG, FB3 to FB3_LCD, FB4 to FB4_LCD, R1 to R1_LED, R10 to R10_CH, R2 to R2_LED, R3 to R3_LED, R34 to R34_FG, R35 to R35_FG, R36 to R36_FG, R37 to R37_FG, R4 to R4_GPS, R7 to R7_FG, R8 to R8_FG
