File: EAGLE/project/FitnessBand/fitnessband.sch (EAGLE design)
At the start: 59 parts, among them J5 TC2030-JLINK-NL, U17 NRF51822QF, X3 EPSON-FA-128, X4 ABS05-32.768KHZ-T, X5 USB-MICROB

Commit message: asdf
Connections:
- net ALT_FG: now also U17.P12; no longer U17.P13
- net QST_FG: now also U17.P13; no longer U17.P12
Changed lines of the file:
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@@
 <?xml version="1.0" encoding="utf-8"?>
 <!DOCTYPE eagle SYSTEM "eagle.dtd">
-<eagle version="6.6.0">
+<eagle version="7.4.0">
 <drawing>
 <settings>
@@
 </segment>
 </net>
-<net name="QST_FG" class="0">
+<net name="ALT_FG" class="0">
 <segment>
 <pinref part="U17" gate="G$1" pin="P12"/>
@@
 </segment>
 </net>
-<net name="ALT_FG" class="0">
+<net name="SCLK_LCD" class="0">
+<segment>
+<pinref part="U17" gate="G$1" pin="P05/AIN6"/>
+<wire x1="15.24" y1="30.48" x2="7.62" y2="30.48" width="0.1524" layer="91"/>
+<label x="-5.08" y="30.48" size="1.778" layer="95"/>
+</segment>
+</net>
+<net name="SI_LCD" class="0">
+<segment>
+<pinref part="U17" gate="G$1" pin="P06/AIN7/AREF1"/>
+<wire x1="15.24" y1="27.94" x2="7.62" y2="27.94" width="0.1524" layer="91"/>
+<label x="-5.08" y="27.94" size="1.778" layer="95"/>
+</segment>
+</net>
+<net name="SCS_LCD" class="0">
+<segment>
+<pinref part="U17" gate="G$1" pin="P07"/>
+<wire x1="15.24" y1="25.4" x2="7.62" y2="25.4" width="0.1524" layer="91"/>
+<label x="-5.08" y="25.4" size="1.778" layer="95"/>
+</segment>
+</net>
+<net name="GPIO1" class="0">
+<segment>
+<pinref part="U17" gate="G$1" pin="P17"/>
+<wire x1="60.96" y1="45.72" x2="68.58" y2="45.72" width="0.1524" layer="91"/>
+<label x="68.58" y="45.72" size="1.778" layer="95"/>
+</segment>
+</net>
+<net name="HR" class="0">
+<segment>
+<pinref part="U17" gate="G$1" pin="P01/AIN2"/>
+<wire x1="15.24" y1="40.64" x2="5.08" y2="40.64" width="0.1524" layer="91"/>
+<label x="2.54" y="38.1" size="1.778" layer="95"/>
+</segment>
+</net>
+<net name="QST_FG" class="0">
 <segment>
 <pinref part="U17" gate="G$1" pin="P13"/>
@@
 </segment>
 </net>
-<net name="SCLK_LCD" class="0">
-<segment>
-<pinref part="U17" gate="G$1" pin="P05/AIN6"/>
-<wire x1="15.24" y1="30.48" x2="7.62" y2="30.48" width="0.1524" layer="91"/>
-<label x="-5.08" y="30.48" size="1.778" layer="95"/>
-</segment>
-</net>
-<net name="SI_LCD" class="0">
-<segment>
-<pinref part="U17" gate="G$1" pin="P06/AIN7/AREF1"/>
-<wire x1="15.24" y1="27.94" x2="7.62" y2="27.94" width="0.1524" layer="91"/>
-<label x="-5.08" y="27.94" size="1.778" layer="95"/>
-</segment>
-</net>
-<net name="SCS_LCD" class="0">
-<segment>
-<pinref part="U17" gate="G$1" pin="P07"/>
-<wire x1="15.24" y1="25.4" x2="7.62" y2="25.4" width="0.1524" layer="91"/>
-<label x="-5.08" y="25.4" size="1.778" layer="95"/>
-</segment>
-</net>
-<net name="GPIO1" class="0">
-<segment>
-<pinref part="U17" gate="G$1" pin="P17"/>
-<wire x1="60.96" y1="45.72" x2="68.58" y2="45.72" width="0.1524" layer="91"/>
-<label x="68.58" y="45.72" size="1.778" layer="95"/>
-</segment>
-</net>
-<net name="HR" class="0">
-<segment>
-<pinref part="U17" gate="G$1" pin="P01/AIN2"/>
-<wire x1="15.24" y1="40.64" x2="5.08" y2="40.64" width="0.1524" layer="91"/>
-<label x="2.54" y="38.1" size="1.778" layer="95"/>
-</segment>
-</net>
