File: EAGLE/project/FitnessBand/fitnessband.sch (EAGLE design)
At the start: 59 parts, among them J5 TC2030-JLINK-NL, U17 NRF51822QF, X3 EPSON-FA-128, X4 ABS05-32.768KHZ-T, X5 USB-MICROB

Commit message: asdf
Parts:
- renumbered B_CONNECTOR to LIPO
Connections:
- net !FRAM_WP: now also U17.P02/AIN3; no longer U17.P16
- net ALT_FG: now also U17.P10; no longer U17.P12
- net BUTTON1: now also U17.P23; no longer U17.P21
- net BUTTON3: now also U17.P21; no longer U17.P23
- net QST_FG: now also U17.P11; no longer U17.P13
- net SCL_FG: now also U17.P12; no longer U17.P11
- net SDA_FG: now also U17.P13; no longer U17.P10
- net SPI_MISO_FRAM: now also U17.P16; no longer U17.P29
- net SPI_MOSI_FRAM: now also U17.P03/AIN4; no longer U17.P30
- net SPI_SCK_FRAM: now also U17.P04/AIN5; no longer U17.P00/AREF0

Commit message: asdf
Parts:
- removed C_FRAM: 0.1uF, resistor:C-EUC0402
- removed FRAM: FM25L04B-DG, chips:FM25L04B-DG
Connections:
- removed net !FRAM_CS: FRAM.!CS, U17.P15
- removed net !FRAM_HOLD: FRAM.!HOLD, U17.P14
- removed net !FRAM_WP: FRAM.!WP, U17.P02/AIN3
- removed net SPI_MISO_FRAM: FRAM.SO, U17.P16
- removed net SPI_MOSI_FRAM: FRAM.SI, U17.P03/AIN4
- removed net SPI_SCK_FRAM: FRAM.SCK, U17.P04/AIN5
- net 3.3V: no longer C_FRAM.1, FRAM.VDD
- net ALT_FG: now also U17.P13; no longer U17.P10
- net GND: no longer C_FRAM.2, FRAM.VSS
- net LED_BLUE: now also U17.P08; no longer U17.P19
- net LED_GREEN: now also U17.P10; no longer U17.P20
- net LED_RED: now also U17.P09; no longer U17.P18
- net QST_FG: now also U17.P14; no longer U17.P11
- net RX_GPS: now also U17.P12; no longer U17.P09
- net SCL_FG: now also U17.P15; no longer U17.P12
- net SDA_FG: now also U17.P16; no longer U17.P13
- net TX_GPS: now also U17.P11; no longer U17.P08
Changed lines of the file:
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@@
 <part name="R2_LED" library="passives" deviceset="RESISTOR" device="0402_RES" value="1k"/>
 <part name="R3_LED" library="passives" deviceset="RESISTOR" device="0402_RES" value="1k"/>
-<part name="GND1" library="supply1" deviceset="GND" device=""/>
-<part name="FRAM" library="chips" deviceset="FM25" device="L04B-DG"/>
-<part name="U$2" library="microbuilder" deviceset="3.3V" device=""/>
 <part name="C2_CH" library="resistor" deviceset="C-EU" device="C0402" value="1uF"/>
 <part name="C3_CH" library="resistor" deviceset="C-EU" device="C0402" value="1uF"/>
 <part name="C4_LDO" library="resistor" deviceset="C-EU" device="C0402"/>
 <part name="C5_GPS" library="resistor" deviceset="C-EU" device="C0402" value="0.1uF"/>
-<part name="C_FRAM" library="resistor" deviceset="C-EU" device="C0402" value="0.1uF"/>
 <part name="C7_IMU" library="resistor" deviceset="C-EU" device="C0402" value="10nF"/>
 <part name="C8_IMU" library="resistor" deviceset="C-EU" device="C0402" value="2.2uF"/>
@@
 <attribute name="VALUE" x="257.81" y="-14.478" size="1.778" layer="96" rot="R180"/>
 </instance>
-<instance part="GND1" gate="1" x="167.64" y="-78.74"/>
-<instance part="FRAM" gate="G$1" x="182.88" y="-68.58"/>
-<instance part="U$2" gate="G$1" x="167.64" y="-55.88"/>
 <instance part="C5_GPS" gate="G$1" x="154.94" y="66.04"/>
-<instance part="C_FRAM" gate="G$1" x="165.1" y="-66.04"/>
 <instance part="C7_IMU" gate="G$1" x="99.06" y="-38.1"/>
 <instance part="C8_IMU" gate="G$1" x="43.18" y="-35.56"/>
@@
 </segment>
 <segment>
-<wire x1="170.18" y1="-73.66" x2="167.64" y2="-73.66" width="0.1524" layer="91"/>
-<wire x1="167.64" y1="-73.66" x2="165.1" y2="-73.66" width="0.1524" layer="91"/>
-<wire x1="165.1" y1="-73.66" x2="165.1" y2="-71.12" width="0.1524" layer="91"/>
-<pinref part="GND1" gate="1" pin="GND"/>
-<wire x1="167.64" y1="-76.2" x2="167.64" y2="-73.66" width="0.1524" layer="91"/>
-<junction x="167.64" y="-73.66"/>
-<pinref part="FRAM" gate="G$1" pin="VSS"/>
-<pinref part="C_FRAM" gate="G$1" pin="2"/>
-</segment>
-<segment>
 <pinref part="U$30" gate="G$1" pin="GND"/>
 <pinref part="JP16" gate="G$1" pin="9"/>
@@
 </segment>
 <segment>
-<wire x1="165.1" y1="-63.5" x2="165.1" y2="-60.96" width="0.1524" layer="91"/>
-<wire x1="165.1" y1="-60.96" x2="167.64" y2="-60.96" width="0.1524" layer="91"/>
-<pinref part="FRAM" gate="G$1" pin="VDD"/>
-<pinref part="U$2" gate="G$1" pin="3.3V"/>
-<wire x1="167.64" y1="-60.96" x2="170.18" y2="-60.96" width="0.1524" layer="91"/>
-<wire x1="167.64" y1="-58.42" x2="167.64" y2="-60.96" width="0.1524" layer="91"/>
-<junction x="167.64" y="-60.96"/>
-<pinref part="C_FRAM" gate="G$1" pin="1"/>
-</segment>
-<segment>
 <pinref part="U$5" gate="G$1" pin="3.3V"/>
 <wire x1="203.2" y1="-17.78" x2="203.2" y2="-20.32" width="0.1524" layer="91"/>
@@
 <wire x1="246.38" y1="-22.86" x2="248.92" y2="-22.86" width="0.1524" layer="91"/>
 <pinref part="R2_LED" gate="G$1" pin="2"/>
-</segment>
-</net>
-<net name="!FRAM_CS" class="0">
-<segment>
-<wire x1="195.58" y1="-71.12" x2="198.12" y2="-71.12" width="0.1524" layer="91"/>
-<label x="198.12" y="-71.12" size="1.27" layer="95" xref="yes"/>
-<pinref part="FRAM" gate="G$1" pin="!CS"/>
-</segment>
-</net>
-<net name="!FRAM_HOLD" class="0">
-<segment>
-<wire x1="195.58" y1="-76.2" x2="198.12" y2="-76.2" width="0.1524" layer="91"/>
-<label x="198.12" y="-76.2" size="1.27" layer="95" xref="yes"/>
-<pinref part="FRAM" gate="G$1" pin="!HOLD"/>
-</segment>
-</net>
-<net name="!FRAM_WP" class="0">
-<segment>
-<wire x1="195.58" y1="-78.74" x2="198.12" y2="-78.74" width="0.1524" layer="91"/>
-<label x="198.12" y="-78.74" size="1.27" layer="95" xref="yes"/>
-<pinref part="FRAM" gate="G$1" pin="!WP"/>
-</segment>
-</net>
-<net name="SPI_SCK_FRAM" class="0">
-<segment>
-<wire x1="195.58" y1="-68.58" x2="198.12" y2="-68.58" width="0.1524" layer="91"/>
-<label x="198.12" y="-68.58" size="1.27" layer="95" xref="yes"/>
-<pinref part="FRAM" gate="G$1" pin="SCK"/>
-</segment>
-</net>
-<net name="SPI_MOSI_FRAM" class="0">
-<segment>
-<wire x1="195.58" y1="-63.5" x2="198.12" y2="-63.5" width="0.1524" layer="91"/>
-<label x="198.12" y="-63.5" size="1.27" layer="95" xref="yes"/>
-<pinref part="FRAM" gate="G$1" pin="SI"/>
-</segment>
-</net>
-<net name="SPI_MISO_FRAM" class="0">
-<segment>
-<wire x1="195.58" y1="-66.04" x2="198.12" y2="-66.04" width="0.1524" layer="91"/>
-<label x="198.12" y="-66.04" size="1.27" layer="95" xref="yes"/>
-<pinref part="FRAM" gate="G$1" pin="SO"/>
 </segment>
 </net>
@@
 </segment>
 </net>
-<net name="SPI_SCK_FRAM" class="0">
-<segment>
-<pinref part="U17" gate="G$1" pin="P04/AIN5"/>
-<wire x1="15.24" y1="33.02" x2="10.16" y2="33.02" width="0.1524" layer="91"/>
-<label x="-5.08" y="33.02" size="1.778" layer="95"/>
-</segment>
-</net>
-<net name="LED_BLUE" class="0">
-<segment>
-<label x="66.04" y="40.64" size="1.27" layer="95" xref="yes"/>
-<pinref part="U17" gate="G$1" pin="P19"/>
-<wire x1="66.04" y1="40.64" x2="60.96" y2="40.64" width="0.1524" layer="91"/>
-</segment>
-</net>
-<net name="LED_GREEN" class="0">
-<segment>
-<label x="66.04" y="38.1" size="1.27" layer="95" xref="yes"/>
-<pinref part="U17" gate="G$1" pin="P20"/>
-<wire x1="60.96" y1="38.1" x2="66.04" y2="38.1" width="0.1524" layer="91"/>
-</segment>
-</net>
-<net name="LED_RED" class="0">
-<segment>
-<label x="66.04" y="43.18" size="1.27" layer="95" xref="yes"/>
-<pinref part="U17" gate="G$1" pin="P18"/>
-<wire x1="60.96" y1="43.18" x2="66.04" y2="43.18" width="0.1524" layer="91"/>
-</segment>
-</net>
-<net name="SPI_MOSI_FRAM" class="0">
-<segment>
-<pinref part="U17" gate="G$1" pin="P03/AIN4"/>
-<wire x1="15.24" y1="35.56" x2="5.08" y2="35.56" width="0.1524" layer="91"/>
-<label x="-5.08" y="35.56" size="1.778" layer="95"/>
-</segment>
-</net>
-<net name="SPI_MISO_FRAM" class="0">
-<segment>
-<label x="66.04" y="48.26" size="1.27" layer="95" xref="yes"/>
-<pinref part="U17" gate="G$1" pin="P16"/>
-<wire x1="66.04" y1="48.26" x2="60.96" y2="48.26" width="0.1524" layer="91"/>
-</segment>
-</net>
 <net name="N$29" class="0">
 <segment>
@@
 <net name="TX_GPS" class="0">
 <segment>
-<pinref part="U17" gate="G$1" pin="P08"/>
-<wire x1="15.24" y1="20.32" x2="7.62" y2="20.32" width="0.1524" layer="91"/>
-<label x="-2.54" y="20.32" size="1.778" layer="95"/>
+<pinref part="U17" gate="G$1" pin="P11"/>
+<wire x1="15.24" y1="12.7" x2="10.16" y2="12.7" width="0.1524" layer="91"/>
+<label x="2.54" y="12.7" size="1.778" layer="95"/>
 </segment>
 </net>
 <net name="RX_GPS" class="0">
 <segment>
-<pinref part="U17" gate="G$1" pin="P09"/>
-<wire x1="15.24" y1="17.78" x2="7.62" y2="17.78" width="0.1524" layer="91"/>
-<label x="-2.54" y="17.78" size="1.778" layer="95"/>
+<pinref part="U17" gate="G$1" pin="P12"/>
+<wire x1="15.24" y1="10.16" x2="10.16" y2="10.16" width="0.1524" layer="91"/>
+<label x="2.54" y="10.16" size="1.778" layer="95"/>
 </segment>
 </net>
@@
 <net name="ALT_FG" class="0">
 <segment>
-<pinref part="U17" gate="G$1" pin="P10"/>
-<wire x1="15.24" y1="15.24" x2="7.62" y2="15.24" width="0.1524" layer="91"/>
-<label x="-2.54" y="15.24" size="1.778" layer="95"/>
+<pinref part="U17" gate="G$1" pin="P13"/>
+<wire x1="15.24" y1="7.62" x2="10.16" y2="7.62" width="0.1524" layer="91"/>
+<label x="2.54" y="7.62" size="1.778" layer="95"/>
 </segment>
 </net>
@@
 <net name="SCL_FG" class="0">
 <segment>
-<pinref part="U17" gate="G$1" pin="P12"/>
-<wire x1="15.24" y1="10.16" x2="7.62" y2="10.16" width="0.1524" layer="91"/>
-<label x="-2.54" y="10.16" size="1.778" layer="95"/>
+<pinref part="U17" gate="G$1" pin="P15"/>
+<wire x1="15.24" y1="2.54" x2="10.16" y2="2.54" width="0.1524" layer="91"/>
+<label x="2.54" y="2.54" size="1.778" layer="95"/>
 </segment>
 </net>
 <net name="SDA_FG" class="0">
 <segment>
-<pinref part="U17" gate="G$1" pin="P13"/>
-<wire x1="15.24" y1="7.62" x2="7.62" y2="7.62" width="0.1524" layer="91"/>
-<label x="-2.54" y="7.62" size="1.778" layer="95"/>
+<pinref part="U17" gate="G$1" pin="P16"/>
+<wire x1="60.96" y1="48.26" x2="68.58" y2="48.26" width="0.1524" layer="91"/>
+<label x="66.04" y="48.26" size="1.778" layer="95"/>
 </segment>
 </net>
 <net name="QST_FG" class="0">
 <segment>
-<pinref part="U17" gate="G$1" pin="P11"/>
-<wire x1="15.24" y1="12.7" x2="7.62" y2="12.7" width="0.1524" layer="91"/>
-<label x="-2.54" y="12.7" size="1.778" layer="95"/>
-</segment>
-</net>
-<net name="!FRAM_HOLD" class="0">
-<segment>
-<label x="7.62" y="5.08" size="1.27" layer="95" rot="R180" xref="yes"/>
 <pinref part="U17" gate="G$1" pin="P14"/>
-<wire x1="7.62" y1="5.08" x2="15.24" y2="5.08" width="0.1524" layer="91"/>
-</segment>
-</net>
-<net name="!FRAM_WP" class="0">
-<segment>
-<pinref part="U17" gate="G$1" pin="P02/AIN3"/>
-<wire x1="15.24" y1="38.1" x2="7.62" y2="38.1" width="0.1524" layer="91"/>
-<label x="-5.08" y="38.1" size="1.778" layer="95"/>
-</segment>
-</net>
-<net name="!FRAM_CS" class="0">
-<segment>
-<label x="7.62" y="2.54" size="1.27" layer="95" rot="R180" xref="yes"/>
-<pinref part="U17" gate="G$1" pin="P15"/>
-<wire x1="7.62" y1="2.54" x2="15.24" y2="2.54" width="0.1524" layer="91"/>
+<wire x1="15.24" y1="5.08" x2="10.16" y2="5.08" width="0.1524" layer="91"/>
+<label x="2.54" y="5.08" size="1.778" layer="95"/>
 </segment>
 </net>
@@
 </segment>
 </net>
+<net name="LED_BLUE" class="0">
+<segment>
+<pinref part="U17" gate="G$1" pin="P08"/>
+<wire x1="15.24" y1="20.32" x2="10.16" y2="20.32" width="0.1524" layer="91"/>
+<label x="-2.54" y="20.32" size="1.778" layer="95"/>
+</segment>
+</net>
+<net name="LED_GREEN" class="0">
+<segment>
+<pinref part="U17" gate="G$1" pin="P10"/>
+<wire x1="15.24" y1="15.24" x2="10.16" y2="15.24" width="0.1524" layer="91"/>
+<label x="-2.54" y="15.24" size="1.778" layer="95"/>
+</segment>
+</net>
+<net name="LED_RED" class="0">
+<segment>
+<pinref part="U17" gate="G$1" pin="P09"/>
+<wire x1="15.24" y1="17.78" x2="10.16" y2="17.78" width="0.1524" layer="91"/>
+<label x="-2.54" y="17.78" size="1.778" layer="95"/>
+</segment>
+</net>

Commit message: no airwires or drc errors
Connections:
- net 3.3V: now also IMU.AD0
- net ALT_FG: now also U17.P16; no longer U17.P13
- net CHARGING?: now also U17.P20
- net GND: no longer IMU.AD0
- net QST_FG: now also U17.P15; no longer U17.P14
- net SCL_FG: now also U17.P14; no longer U17.P15
- net SDA_FG: now also U17.P13; no longer U17.P16
Changed lines of the file:
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@@
 <part name="GND70" library="SparkFun" deviceset="GND" device=""/>
 <part name="GND71" library="SparkFun" deviceset="GND" device=""/>
-<part name="GND73" library="SparkFun" deviceset="GND" device=""/>
 <part name="GND74" library="SparkFun" deviceset="GND" device=""/>
 <part name="U$89" library="microbuilder" deviceset="3.3V" device=""/>
@@
 <part name="U$5" library="microbuilder" deviceset="3.3V" device=""/>
 <part name="U$6" library="microbuilder" deviceset="3.3V" device=""/>
+<part name="U$2" library="microbuilder" deviceset="3.3V" device=""/>
 </parts>
 <sheets>
@@
 <instance part="GND70" gate="1" x="35.56" y="-45.72"/>
 <instance part="GND71" gate="1" x="27.94" y="-33.02"/>
-<instance part="GND73" gate="1" x="111.76" y="-33.02"/>
 <instance part="GND74" gate="1" x="20.32" y="-33.02"/>
 <instance part="U$89" gate="G$1" x="48.26" y="2.54"/>
@@
 <instance part="U$5" gate="G$1" x="203.2" y="-15.24"/>
 <instance part="U$6" gate="G$1" x="220.98" y="-10.16"/>
+<instance part="U$2" gate="G$1" x="119.38" y="-33.02"/>
 </instances>
 <busses>
@@
 </segment>
 <segment>
-<pinref part="GND73" gate="1" pin="GND"/>
-<wire x1="111.76" y1="-30.48" x2="111.76" y2="-27.94" width="0.1524" layer="91"/>
-<pinref part="IMU" gate="G$1" pin="AD0"/>
-<wire x1="111.76" y1="-27.94" x2="88.9" y2="-27.94" width="0.1524" layer="91"/>
-</segment>
-<segment>
 <label x="45.72" y="-22.86" size="1.778" layer="95"/>
 <pinref part="IMU" gate="G$1" pin="FSYNC"/>
@@
 <pinref part="RGB_LED" gate="G$1" pin="VDD"/>
 <wire x1="220.98" y1="-17.78" x2="223.52" y2="-17.78" width="0.1524" layer="91"/>
+</segment>
+<segment>
+<pinref part="U$2" gate="G$1" pin="3.3V"/>
+<wire x1="119.38" y1="-35.56" x2="119.38" y2="-38.1" width="0.1524" layer="91"/>
+<wire x1="119.38" y1="-38.1" x2="111.76" y2="-38.1" width="0.1524" layer="91"/>
+<pinref part="IMU" gate="G$1" pin="AD0"/>
+<wire x1="111.76" y1="-27.94" x2="88.9" y2="-27.94" width="0.1524" layer="91"/>
+<wire x1="111.76" y1="-38.1" x2="111.76" y2="-27.94" width="0.1524" layer="91"/>
 </segment>
 </net>
@@
 </segment>
 </net>
-<net name="ALT_FG" class="0">
+<net name="SCLK_LCD" class="0">
+<segment>
+<pinref part="U17" gate="G$1" pin="P05/AIN6"/>
+<wire x1="15.24" y1="30.48" x2="7.62" y2="30.48" width="0.1524" layer="91"/>
+<label x="-5.08" y="30.48" size="1.778" layer="95"/>
+</segment>
+</net>
+<net name="SI_LCD" class="0">
+<segment>
+<pinref part="U17" gate="G$1" pin="P06/AIN7/AREF1"/>
+<wire x1="15.24" y1="27.94" x2="7.62" y2="27.94" width="0.1524" layer="91"/>
+<label x="-5.08" y="27.94" size="1.778" layer="95"/>
+</segment>
+</net>
+<net name="SCS_LCD" class="0">
+<segment>
+<pinref part="U17" gate="G$1" pin="P07"/>
+<wire x1="15.24" y1="25.4" x2="7.62" y2="25.4" width="0.1524" layer="91"/>
+<label x="-5.08" y="25.4" size="1.778" layer="95"/>
+</segment>
+</net>
+<net name="GPIO1" class="0">
+<segment>
+<pinref part="U17" gate="G$1" pin="P17"/>
+<wire x1="60.96" y1="45.72" x2="68.58" y2="45.72" width="0.1524" layer="91"/>
+<label x="68.58" y="45.72" size="1.778" layer="95"/>
+</segment>
+</net>
+<net name="HR" class="0">
+<segment>
+<pinref part="U17" gate="G$1" pin="P01/AIN2"/>
+<wire x1="15.24" y1="40.64" x2="5.08" y2="40.64" width="0.1524" layer="91"/>
+<label x="5.08" y="40.64" size="1.778" layer="95"/>
+</segment>
+</net>
+<net name="SCL_FG" class="0">
+<segment>
+<pinref part="U17" gate="G$1" pin="P14"/>
+<wire x1="15.24" y1="5.08" x2="10.16" y2="5.08" width="0.1524" layer="91"/>
+<label x="2.54" y="5.08" size="1.778" layer="95"/>
+</segment>
+</net>
+<net name="SDA_FG" class="0">
 <segment>
 <pinref part="U17" gate="G$1" pin="P13"/>
@@
 </segment>
 </net>
-<net name="SCLK_LCD" class="0">
-<segment>
-<pinref part="U17" gate="G$1" pin="P05/AIN6"/>
-<wire x1="15.24" y1="30.48" x2="7.62" y2="30.48" width="0.1524" layer="91"/>
-<label x="-5.08" y="30.48" size="1.778" layer="95"/>
-</segment>
-</net>
-<net name="SI_LCD" class="0">
-<segment>
-<pinref part="U17" gate="G$1" pin="P06/AIN7/AREF1"/>
-<wire x1="15.24" y1="27.94" x2="7.62" y2="27.94" width="0.1524" layer="91"/>
-<label x="-5.08" y="27.94" size="1.778" layer="95"/>
-</segment>
-</net>
-<net name="SCS_LCD" class="0">
-<segment>
-<pinref part="U17" gate="G$1" pin="P07"/>
-<wire x1="15.24" y1="25.4" x2="7.62" y2="25.4" width="0.1524" layer="91"/>
-<label x="-5.08" y="25.4" size="1.778" layer="95"/>
-</segment>
-</net>
-<net name="GPIO1" class="0">
-<segment>
-<pinref part="U17" gate="G$1" pin="P17"/>
-<wire x1="60.96" y1="45.72" x2="68.58" y2="45.72" width="0.1524" layer="91"/>
-<label x="68.58" y="45.72" size="1.778" layer="95"/>
-</segment>
-</net>
-<net name="HR" class="0">
-<segment>
-<pinref part="U17" gate="G$1" pin="P01/AIN2"/>
-<wire x1="15.24" y1="40.64" x2="5.08" y2="40.64" width="0.1524" layer="91"/>
-<label x="5.08" y="40.64" size="1.778" layer="95"/>
-</segment>
-</net>
-<net name="SCL_FG" class="0">
+<net name="BUTTON1" class="0">
+<segment>
+<pinref part="U17" gate="G$1" pin="P23"/>
+<wire x1="60.96" y1="30.48" x2="66.04" y2="30.48" width="0.1524" layer="91"/>
+<label x="66.04" y="30.48" size="1.778" layer="95"/>
+</segment>
+</net>
+<net name="LED_BLUE" class="0">
+<segment>
+<pinref part="U17" gate="G$1" pin="P08"/>
+<wire x1="15.24" y1="20.32" x2="10.16" y2="20.32" width="0.1524" layer="91"/>
+<label x="-2.54" y="20.32" size="1.778" layer="95"/>
+</segment>
+</net>
+<net name="LED_GREEN" class="0">
+<segment>
+<pinref part="U17" gate="G$1" pin="P10"/>
+<wire x1="15.24" y1="15.24" x2="10.16" y2="15.24" width="0.1524" layer="91"/>
+<label x="-2.54" y="15.24" size="1.778" layer="95"/>
+</segment>
+</net>
+<net name="LED_RED" class="0">
+<segment>
+<pinref part="U17" gate="G$1" pin="P09"/>
+<wire x1="15.24" y1="17.78" x2="10.16" y2="17.78" width="0.1524" layer="91"/>
+<label x="-2.54" y="17.78" size="1.778" layer="95"/>
+</segment>
+</net>
+<net name="ALT_FG" class="0">
+<segment>
+<pinref part="U17" gate="G$1" pin="P16"/>
+<wire x1="60.96" y1="48.26" x2="68.58" y2="48.26" width="0.1524" layer="91"/>
+<label x="66.04" y="48.26" size="1.778" layer="95"/>
+</segment>
+</net>
+<net name="QST_FG" class="0">
 <segment>
 <pinref part="U17" gate="G$1" pin="P15"/>
@@
 </segment>
 </net>
-<net name="SDA_FG" class="0">
-<segment>
-<pinref part="U17" gate="G$1" pin="P16"/>
-<wire x1="60.96" y1="48.26" x2="68.58" y2="48.26" width="0.1524" layer="91"/>
-<label x="66.04" y="48.26" size="1.778" layer="95"/>
-</segment>
-</net>
-<net name="QST_FG" class="0">
-<segment>
-<pinref part="U17" gate="G$1" pin="P14"/>
-<wire x1="15.24" y1="5.08" x2="10.16" y2="5.08" width="0.1524" layer="91"/>
-<label x="2.54" y="5.08" size="1.778" layer="95"/>
-</segment>
-</net>
-<net name="BUTTON1" class="0">
-<segment>
-<pinref part="U17" gate="G$1" pin="P23"/>
-<wire x1="60.96" y1="30.48" x2="66.04" y2="30.48" width="0.1524" layer="91"/>
-<label x="66.04" y="30.48" size="1.778" layer="95"/>
-</segment>
-</net>
-<net name="LED_BLUE" class="0">
-<segment>
-<pinref part="U17" gate="G$1" pin="P08"/>
-<wire x1="15.24" y1="20.32" x2="10.16" y2="20.32" width="0.1524" layer="91"/>
-<label x="-2.54" y="20.32" size="1.778" layer="95"/>
-</segment>
-</net>
-<net name="LED_GREEN" class="0">
-<segment>
-<pinref part="U17" gate="G$1" pin="P10"/>
-<wire x1="15.24" y1="15.24" x2="10.16" y2="15.24" width="0.1524" layer="91"/>
-<label x="-2.54" y="15.24" size="1.778" layer="95"/>
-</segment>
-</net>
-<net name="LED_RED" class="0">
-<segment>
-<pinref part="U17" gate="G$1" pin="P09"/>
-<wire x1="15.24" y1="17.78" x2="10.16" y2="17.78" width="0.1524" layer="91"/>
-<label x="-2.54" y="17.78" size="1.778" layer="95"/>
-</segment>
-</net>
+<net name="CHARGING?" class="0">
+<segment>
+<pinref part="U17" gate="G$1" pin="P20"/>
+<wire x1="60.96" y1="38.1" x2="66.04" y2="38.1" width="0.1524" layer="91"/>
+<label x="66.04" y="38.1" size="1.778" layer="95"/>
+</segment>
+</net>

Commit message: changes from rev2
Connections:
- net SCL_IMU: now also U17.P25; no longer U17.P24
- net SDA_IMU: now also U17.P24; no longer U17.P25
Changed lines of the file:
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@@
 </segment>
 </net>
-<net name="SCL_IMU" class="0">
+<net name="SDA_IMU" class="0">
 <segment>
 <pinref part="U17" gate="G$1" pin="P24"/>
 <wire x1="60.96" y1="25.4" x2="66.04" y2="25.4" width="0.1524" layer="91"/>
 <label x="66.04" y="25.4" size="1.778" layer="95"/>
-</segment>
-</net>
-<net name="SDA_IMU" class="0">
-<segment>
-<pinref part="U17" gate="G$1" pin="P25"/>
-<wire x1="60.96" y1="22.86" x2="66.04" y2="22.86" width="0.1524" layer="91"/>
-<label x="66.04" y="22.86" size="1.778" layer="95"/>
 </segment>
 </net>
@@
 </segment>
 </net>
+<net name="SCL_IMU" class="0">
+<segment>
+<pinref part="U17" gate="G$1" pin="P25"/>
+<wire x1="60.96" y1="22.86" x2="66.04" y2="22.86" width="0.1524" layer="91"/>
+<label x="66.04" y="22.86" size="1.778" layer="95"/>
+</segment>
+</net>
