File: EAGLE/project/FitnessBand/fitnessband.brd (EAGLE design)
At the start: 35.2 x 27.9 mm, 59 parts, among them J5 TC2030-JLINK-NL, U17 NRF51822QF, X3 EPSON-FA-128, X4 ABS05-32.768KHZ-T, X5 USB-MICROB

Commit message: began layot
Parts:
- removed C2, C3: 1uF, resistor:C0402
- removed C4: (no value), resistor:C0402
- removed C5: 0.1uF, resistor:C0402
- removed C62: 1uF, SparkFun:0402-CAP
- removed C63: 10nF, SparkFun:0402-CAP
- removed FB3, FB4: (no value), microbuilder:_0805
- removed R10: 100K, resistor:R0402
- removed R34, R35, R36, R37: 4.7k, SparkFun:0402-RES
- removed R4: 1K, resistor:R0402
- removed R7: 1k, SparkFun:0402-RES
- removed R8: 180, SparkFun:0402-RES
- added C2_CH, C3_CH: 1uF, resistor:C0402
- added C4_LDO: (no value), resistor:C0402
- added C5_GPS: 0.1uF, resistor:C0402
- added C62_FG: 1uF, SparkFun:0402-CAP
- added C63_FG: 10nF, SparkFun:0402-CAP
- added FB3_LCD, FB4_LCD: (no value), microbuilder:_0805
- added R10_CH: 100K, resistor:R0402
- added R34_FG, R35_FG, R36_FG, R37_FG: 4.7k, SparkFun:0402-RES
- added R4_GPS: 1K, resistor:R0402
- added R7_FG: 1k, SparkFun:0402-RES
- added R8_FG: 180, SparkFun:0402-RES
- moved C47 89.8 mm to (20.2, 17.5)
- moved C15_LCD 84.0 mm to (20.6, 21.1), flipped to the bottom, turned to 180 degrees
- moved C14_LCD 81.1 mm to (23.1, 22.4), flipped to the bottom, turned to 180 degrees
- moved C56 80.2 mm to (17.9, 24.5), turned to 90 degrees
- moved C59 79.0 mm to (29.1, 27.2), turned to 180 degrees
- moved C58 77.3 mm to (30.9, 21.1), turned to 270 degrees
- moved C55 76.3 mm to (18.7, 24.5), turned to 90 degrees
- moved C53 74.2 mm to (30.5, 19.9)
- moved C50 74.2 mm to (24.3, 18.4), turned to 270 degrees
- moved C57 73.0 mm to (21.2, 21.6), turned to 90 degrees
- moved C52 71.3 mm to (30.5, 18.1)
- moved C16_LCD 64.7 mm to (17.3, 22.7), flipped to the bottom
- moved X4 64.5 mm to (30.4, 19.0)
- moved C48 58.5 mm to (23.0, 18.0)
- moved C49 55.2 mm to (20.0, 24.5), turned to 180 degrees
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- renumbered R1 to R1_LED, R2 to R2_LED, R3 to R3_LED
Connections:
- net 3.3V: now also C4_LDO.1, C5_GPS.1, FB3_LCD.1, R10_CH.2, R34_FG.2, R36_FG.2, R37_FG.2; no longer C4.1, C5.1, FB3.1, R10.2, R34.2, R36.2, R37.2
- net AGLCD: now also FB4_LCD.2; no longer FB4.2
- net ALCD: now also FB3_LCD.2; no longer FB3.2
- net ALT_FG: now also R34_FG.1; no longer R34.1
- net BATTERY: now also C3_CH.1, R7_FG.1, R8_FG.2; no longer C3.1, R7.1, R8.2
- net CHARGING?: now also R10_CH.1; no longer R10.1
- net GND: now also C2_CH.2, C3_CH.2, C4_LDO.2, C5_GPS.2, C62_FG.2, C63_FG.2, FB4_LCD.1, R35_FG.1, R4_GPS.1; no longer C2.2, C3.2, C4.2, C5.2, C62.2, C63.2, FB4.1, R35.1, R4.1
- net N$23: now also R4_GPS.2; no longer R4.2
- net N$47: now also C62_FG.1, R7_FG.2; no longer C62.1, R7.2
- net QST_FG: now also R35_FG.2; no longer R35.2
- net SCL_FG: now also R36_FG.1; no longer R36.1
- net SDA_FG: now also R37_FG.1; no longer R37.1
- net USB_PORT: now also C2_CH.1; no longer C2.1
- net VDD: now also C63_FG.1, R8_FG.1; no longer C63.1, R8.1
Routing:
- net SDA_FG: track 0.00 -> 43.2 mm, vias 0 -> 2
- net 3.3V: track 0.00 -> 32.5 mm, vias 0 -> 6
- net AGLCD: track 0.00 -> 11.4 mm
- net N$29: track 0.00 -> 5.83 mm
- net ALCD: track 0.00 -> 5.79 mm
- net N$28: track 0.00 -> 5.08 mm
- net N$35: track 0.00 -> 4.17 mm
- net VDD: track 0.00 -> 4.01 mm
- net N$26: track 0.00 -> 3.82 mm
- net ANTENNA1: track 0.00 -> 3.36 mm
- net N$33: track 0.00 -> 2.91 mm
- net N$34: track 0.00 -> 2.89 mm
- net QST_FG: track 0.00 -> 2.88 mm
- net N$25: track 0.00 -> 2.85 mm
- net GND: track 0.00 -> 2.80 mm
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- added copper zone on layer 15, net 3.3V
- added copper zone on layer 1, net GND
- added copper zone on layer 16, net GND
- added copper zone on layer 16, net N$6
Other:
- board size 35.2 x 27.9 mm -> 40 x 30.1 mm

Commit message: asdf
Parts:
- moved LED1 91.7 mm to (44.2, 7.73)
- moved R1_LED 91.7 mm to (30.2, 12.8)
- moved R3_LED 91.7 mm to (22.6, 12.8)
- moved R2_LED 91.7 mm to (26.4, 12.8)
- moved R4_GPS 86.5 mm to (29.7, 4.16)
- moved C7_IMU 84.8 mm to (31.1, 20.5), turned to 180 degrees
- moved RGB_LED 80.3 mm to (25.7, 3.61)
- moved C13_IMU 76.8 mm to (36.5, 22.8), turned to 270 degrees
- moved R9_IMU 74.2 mm to (28.6, 27.1), turned to 180 degrees
- moved R5_IMU 72.0 mm to (28.6, 28.7), turned to 180 degrees
- moved C12_IMU 69.7 mm to (34.5, 20.5)
- moved R25 62.3 mm to (9.51, 28.9)
- moved C8_IMU 59.2 mm to (32.5, 28.7), turned to 180 degrees
- moved C_FRAM 25.9 mm to (2.10, 29.2)
- moved IMU 24.1 mm to (33.2, 24.5)
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Connections:
- net ALT_FG: now also U17.18; no longer U17.19
- net QST_FG: now also U17.19; no longer U17.18
Routing:
- net SDA_FG: track 43.2 -> 3.56 mm, vias 2 -> 0
- net RX_GPS: track 0.00 -> 34.0 mm, vias 0 -> 2
- net TX_GPS: track 0.00 -> 33.8 mm, vias 0 -> 2
- net SCL_IMU: track 0.00 -> 29.1 mm
- net !FRAM_CS: track 0.00 -> 23.3 mm, vias 0 -> 2
- net SPI_MISO_FRAM: track 0.00 -> 17.2 mm, vias 0 -> 2
- net 3.3V: track 32.5 -> 39.4 mm, vias 6 -> 9
- net BUTTON2: track 0.00 -> 5.02 mm
- net SDA_IMU: track 0.00 -> 3.26 mm
- net VDD: track 4.01 -> 7.08 mm, vias 0 -> 2
- net N$48: track 0.00 -> 2.70 mm
- net N$47: track 1.56 -> 4.01 mm
- net N$49: track 0.00 -> 2.02 mm

Commit message: asdf
Parts:
- moved X5 23.7 mm to (-4.54, 28.1)
- moved GPS 11.4 mm to (37.7, 3.54)
- moved C5_GPS 10.6 mm to (27.2, 8.11)
- moved B_CONNECTOR 9.25 mm to (3.83, 5.10)
- moved FRAM 7.92 mm to (19.1, 7.62)
- moved C59 3.90 mm to (18.4, 24.6), turned to 90 degrees
- moved R25 3.76 mm to (10.6, 25.4)
- moved C58 3.24 mm to (20.0, 19.2)
- moved C48 3.24 mm to (12.1, 16.1)
- moved C57 3.24 mm to (10.3, 19.7)
- moved C49 3.24 mm to (9.05, 22.6)
- moved BALUN 3.24 mm to (7.89, 21.3)
- moved C50 3.24 mm to (13.4, 16.5)
- moved C53 3.24 mm to (19.6, 18.1)
- moved C55 3.24 mm to (7.84, 22.6)
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Routing:
- net 3.3V: track 39.4 -> 67.8 mm
- net RX_GPS: track 34.0 -> 6.00 mm, vias 2 -> 1
- net TX_GPS: track 33.8 -> 14.6 mm
- net SCL_IMU: track 29.1 -> 11.0 mm
- net SPI_MISO_FRAM: track 17.2 -> 0.00 mm, vias 2 -> 0
- net !FRAM_CS: track 23.3 -> 10.7 mm, vias 2 -> 1
- net !FRAM_WP: track 0.00 -> 9.06 mm, vias 0 -> 1
- net SCL_FG: track 2.70 -> 11.2 mm, vias 0 -> 1
- net SDA_FG: track 3.56 -> 10.8 mm, vias 0 -> 1
- net SWDIO/!RESET: track 0.00 -> 7.12 mm, vias 0 -> 1
- net SCLK_LCD: track 0.00 -> 5.31 mm, vias 0 -> 1
- net SI_LCD: track 0.00 -> 4.05 mm, vias 0 -> 1
- net BUTTON2: track 5.02 -> 1.46 mm
- net SCS_LCD: track 0.00 -> 3.21 mm, vias 0 -> 1
- net HR: track 0.00 -> 2.92 mm, vias 0 -> 1
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
Commit message: asdf
Parts:
- removed B_CONNECTOR: SH_MALE_2/1MM, headers:SH-1X2/1MM
- added LIPO: SH_MALE_2/1MM, headers:SH-1X2/1MM
- moved LED1 41.2 mm to (3.75, 15.3), flipped to the bottom, turned to 270 degrees
- moved J5 36.5 mm to (32.9, 3.54), turned to 180 degrees
- moved GPS 33.4 mm to (9.05, 20.7), turned to 90 degrees
- moved R25 31.2 mm to (30.1, 0.98), flipped to the bottom, turned to 180 degrees
- moved R4_GPS 30.6 mm to (2.52, 18.1), flipped to the bottom, turned to 270 degrees
- moved ANT 28.2 mm to (30.7, 6.86), turned to 0 degrees
- moved C47 24.8 mm to (33.7, 11.1), turned to 90 degrees
- moved C5_GPS 24.5 mm to (2.87, 11.2), turned to 180 degrees
- moved C56 24.0 mm to (26.7, 8.81), turned to 180 degrees
- moved X5 23.5 mm to (1.38, 5.36)
- moved BALUN 23.2 mm to (28.0, 9.68), turned to 270 degrees
- moved C55 22.9 mm to (26.7, 9.63), turned to 180 degrees
- moved FRAM 22.8 mm to (4.46, 25.2), flipped to the bottom, turned to 90 degrees
- moved X3 22.3 mm to (32.0, 12.1), turned to 0 degrees
- moved C49 21.2 mm to (26.7, 10.8), turned to 270 degrees
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Connections:
- net !FRAM_WP: now also U17.6; no longer U17.22
- net ALT_FG: now also U17.16; no longer U17.18
- net BATTERY: now also LIPO.2; no longer B_CONNECTOR.2
- net BUTTON1: now also U17.42; no longer U17.40
- net BUTTON3: now also U17.40; no longer U17.42
- net GND: now also LIPO.1; no longer B_CONNECTOR.1
- net QST_FG: now also U17.17; no longer U17.19
- net SCL_FG: now also U17.18; no longer U17.17
- net SDA_FG: now also U17.19; no longer U17.16
- net SPI_MISO_FRAM: now also U17.22; no longer U17.48
- net SPI_MOSI_FRAM: now also U17.7; no longer U17.3
- net SPI_SCK_FRAM: now also U17.8; no longer U17.4
Routing:
- net 3.3V: track 67.8 -> 134.6 mm, vias 9 -> 14
- net !FRAM_WP: track 9.06 -> 38.6 mm
- net SPI_MISO_FRAM: track 0.00 -> 29.3 mm, vias 0 -> 1
- net SPI_MOSI_FRAM: track 1.25 -> 30.0 mm
- net SPI_SCK_FRAM: track 1.92 -> 29.6 mm
- net ALT_FG: track 4.85 -> 29.3 mm, vias 1 -> 2
- net !FRAM_HOLD: track 2.83 -> 24.5 mm
- net QST_FG: track 5.76 -> 27.2 mm, vias 1 -> 2
- net SWDCLK: track 1.47 -> 21.1 mm, vias 0 -> 1
- net BATTERY: track 2.38 -> 20.2 mm, vias 0 -> 1
- net !FRAM_CS: track 10.7 -> 26.4 mm
- net BUTTON1: track 0.00 -> 15.6 mm
- net BUTTON3: track 0.00 -> 15.3 mm
- net SDA_IMU: track 3.26 -> 18.4 mm, vias 0 -> 1
- net SCL_FG: track 11.2 -> 25.3 mm, vias 1 -> 2
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- added copper zone on layer 1, net 3.3V
- added copper zone on layer 16, net 3.3V
- added copper zone on layer 1, net USB_PORT
- removed copper zone on layer 15, net 3.3V
- removed copper zone on layer 16, net N$6

Commit message: asdf
Routing:
- net !FRAM_WP: track 38.6 -> 36.5 mm
Changed lines of the file:
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@@
 <?xml version="1.0" encoding="utf-8"?>
 <!DOCTYPE eagle SYSTEM "eagle.dtd">
-<eagle version="6.6.0">
+<eagle version="7.4.0">
 <drawing>
 <settings>
@@
 <pass name="Default">
 <param name="RoutingGrid" value="50mil"/>
+<param name="AutoGrid" value="1"/>
+<param name="Efforts" value="0"/>
+<param name="TopRouterVariant" value="1"/>
 <param name="tpViaShape" value="round"/>
 <param name="PrefDir.1" value="|"/>
@@
 <wire x1="33.12" y1="21.85306875" x2="31.24" y2="21.84306875" width="0" layer="19" extent="1-1"/>
 <wire x1="34.52" y1="20.02" x2="33.12" y2="21.85306875" width="0" layer="19" extent="1-16"/>
-<wire x1="2.4534" y1="26.615" x2="3.8" y2="28.16" width="0" layer="19" extent="1-16"/>
 <wire x1="33.22" y1="14.36306875" x2="31.285" y2="12.655" width="0" layer="19" extent="1-1"/>
 <wire x1="33.22306875" y1="15.1408" x2="33.22" y2="14.36306875" width="0" layer="19" extent="1-1"/>
@@
 <wire x1="15.03" y1="25.29" x2="14.61" y2="25.29" width="0.1524" layer="16"/>
 <wire x1="14.61" y1="25.29" x2="12.04" y2="27.86" width="0.1524" layer="16"/>
-<wire x1="12.04" y1="27.86" x2="2.23" y2="27.86" width="0.1524" layer="16"/>
-<wire x1="2.23" y1="27.86" x2="1.64" y2="27.27" width="0.1524" layer="16"/>
-<wire x1="1.64" y1="27.27" x2="1.64" y2="25.5284" width="0.1524" layer="16"/>
-<wire x1="1.64" y1="25.5284" x2="2.3168" y2="25.5284" width="0.1524" layer="16"/>
 <wire x1="2.3168" y1="25.5284" x2="2.4534" y2="25.665" width="0.1524" layer="16"/>
+<wire x1="12.04" y1="27.86" x2="3.87" y2="27.86" width="0.1524" layer="16"/>
+<wire x1="3.87" y1="27.86" x2="3.15" y2="27.14" width="0.1524" layer="16"/>
+<wire x1="3.15" y1="27.14" x2="3.15" y2="26.3616" width="0.1524" layer="16"/>
+<wire x1="3.15" y1="26.3616" x2="2.4534" y2="25.665" width="0.1524" layer="16"/>
 </signal>
 <signal name="SPI_SCK_FRAM">

Commit message: asdf
Parts:
- removed C_FRAM: 0.1uF, resistor:C0402
- removed FRAM: FM25L04B-DG, chips:TDFN-8
- moved R3_LED 25.5 mm to (2.39, 23.2), flipped to the bottom, turned to 90 degrees
- moved RGB_LED 25.1 mm to (3.59, 25.3), flipped to the bottom, turned to 270 degrees
- moved R1_LED 24.2 mm to (3.36, 23.2), turned to 90 degrees
- moved R2_LED 23.7 mm to (4.39, 23.2), flipped to the bottom, turned to 90 degrees
Connections:
- removed net !FRAM_CS: FRAM.1, U17.21
- removed net !FRAM_HOLD: FRAM.7, U17.20
- removed net !FRAM_WP: FRAM.3, U17.6
- removed net SPI_MISO_FRAM: FRAM.2, U17.22
- removed net SPI_MOSI_FRAM: FRAM.5, U17.7
- removed net SPI_SCK_FRAM: FRAM.6, U17.8
- net 3.3V: no longer C_FRAM.1, FRAM.8
- net ALT_FG: now also U17.19; no longer U17.16
- net GND: no longer C_FRAM.2, FRAM.4
- net LED_BLUE: now also U17.14; no longer U17.27
- net LED_GREEN: now also U17.16; no longer U17.28
- net LED_RED: now also U17.15; no longer U17.26
- net QST_FG: now also U17.20; no longer U17.17
- net RX_GPS: now also U17.18; no longer U17.15
- net SCL_FG: now also U17.21; no longer U17.18
- net SDA_FG: now also U17.22; no longer U17.19
- net TX_GPS: now also U17.17; no longer U17.14
Routing:
- net !FRAM_WP: track 36.5 -> 0.00 mm, vias 1 -> 0
- net SPI_MOSI_FRAM: track 30.0 -> 0.00 mm, vias 1 -> 0
- net SPI_SCK_FRAM: track 29.6 -> 0.00 mm, vias 1 -> 0
- net SPI_MISO_FRAM: track 29.3 -> 0.00 mm, vias 1 -> 0
- net !FRAM_CS: track 26.4 -> 0.00 mm, vias 1 -> 0
- net LED_GREEN: track 0.00 -> 25.4 mm, vias 0 -> 1
- net LED_RED: track 0.00 -> 24.7 mm, vias 0 -> 1
- net !FRAM_HOLD: track 24.5 -> 0.00 mm, vias 1 -> 0
- net LED_BLUE: track 0.00 -> 23.9 mm, vias 0 -> 1
- net GPIO1: track 0.00 -> 22.7 mm, vias 0 -> 1
- net HR: track 0.00 -> 17.2 mm, vias 0 -> 1
- net GND: track 18.2 -> 28.4 mm, vias 21 -> 24
- net 3.3V: track 134.6 -> 143.9 mm, vias 14 -> 13
- net SWDIO/!RESET: track 18.4 -> 23.1 mm
- net SWDCLK: track 21.1 -> 25.7 mm
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
Commit message: no airwires or drc errors
Parts:
- moved R25 7.11 mm to (36.7, 3.59), turned to 90 degrees
- moved C3_CH 6.13 mm to (11.5, 3.06), turned to 270 degrees
- moved C2_CH 2.58 mm to (5.75, 8.91), turned to 90 degrees
- moved J5 1.12 mm to (32.7, 2.45), turned to 0 degrees
- moved C7_IMU 0.93 mm to (33.7, 24.0)
- moved R10_CH 0.80 mm to (8.31, 3.50)
- moved C16_LCD 0.46 mm to (16.0, 22.8)
- moved C50 0.44 mm to (33.2, 15.2)
- moved C47 0.31 mm to (34.0, 11.1)
- moved X3 0.27 mm to (32.3, 12.1)
- moved R3_LED 0.20 mm to (2.19, 23.2)
- moved CHARGER 0.06 mm to (8.71, 6.00)
- moved C48 0.05 mm to (33.2, 14.0)
Connections:
- net 3.3V: now also IMU.9
- net ALT_FG: now also U17.22; no longer U17.19
- net CHARGING?: now also U17.28
- net GND: no longer IMU.9
- net QST_FG: now also U17.21; no longer U17.20
- net SCL_FG: now also U17.20; no longer U17.21
- net SDA_FG: now also U17.19; no longer U17.22
Routing:
- net 3.3V: track 143.9 -> 194.8 mm, vias 13 -> 9
- net CHARGING?: track 2.33 -> 33.6 mm, vias 0 -> 4
- net GND: track 28.4 -> 42.3 mm, vias 24 -> 34
- net ALT_FG: track 26.6 -> 21.0 mm
- net USB_PORT: track 0.00 -> 4.80 mm
- net SWDCLK: track 25.7 -> 21.8 mm, vias 1 -> 2
- net INT_IMU: track 7.15 -> 10.8 mm
- net SWDIO/!RESET: track 23.1 -> 19.5 mm
- net GPIO1: track 22.7 -> 19.1 mm
- net SCL_FG: track 22.0 -> 18.7 mm
- net QST_FG: track 23.9 -> 20.8 mm
- net SDA_FG: track 20.4 -> 18.0 mm
- net BATTERY: track 20.2 -> 17.9 mm
- net SCLK_LCD: track 17.1 -> 19.4 mm
- net SI_LCD: track 15.6 -> 17.3 mm
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- removed copper zone on layer 1, net 3.3V
- removed copper zone on layer 16, net 3.3V
- removed copper zone on layer 1, net USB_PORT

Commit message: asdf
Parts:
- moved R25 0.90 mm to (36.2, 4.32), turned to 0 degrees
- moved C5_GPS 0.70 mm to (2.18, 11.1)
- moved C14_LCD 0.68 mm to (23.3, 23.0)
- moved C3_CH 0.10 mm to (11.4, 2.97)
Routing:
- net GND: track 42.3 -> 40.6 mm, vias 34 -> 38
- net SWDCLK: track 21.8 -> 20.8 mm
- net CHARGING?: track 33.6 -> 34.3 mm
- net ALCD: track 18.6 -> 17.9 mm
