File: EAGLE/project/FitnessBand/fitnessband.brd (EAGLE design)
At the start: 40 x 30.1 mm, 57 parts, among them J5 TC2030-JLINK-NL, U17 NRF51822QF, X3 EPSON-FA-128, X4 ABS05-32.768KHZ-T, X5 USB-MICROB

Commit message: adc
Parts:
- moved R3_LED 5.04 mm to (6.21, 26.2), turned to 0 degrees
- moved J5 0.09 mm to (32.7, 2.54)
Routing:
- net N$2: track 2.87 -> 5.14 mm
- net 3.3V: track 195.0 -> 196.6 mm
- net LED_GREEN: track 26.0 -> 26.8 mm

Commit message: changes from rev2
Parts:
- moved R9_IMU 9.97 mm to (24.6, 26.8), flipped to the top, turned to 270 degrees
- moved C13_IMU 8.82 mm to (35.3, 26.2)
- moved C7_IMU 6.66 mm to (27.2, 22.6), flipped to the top, turned to 180 degrees
- moved C8_IMU 5.74 mm to (33.8, 27.0), turned to 270 degrees
- moved C12_IMU 2.83 mm to (32.1, 22.2), turned to 180 degrees
- moved R5_IMU 2.27 mm to (32.4, 26.6), turned to 270 degrees
- moved IMU 1.54 mm to (28.8, 26.1), flipped to the top
- moved R3_LED 0.38 mm to (6.24, 26.6)
- moved J5 0.09 mm to (32.7, 2.45)
Connections:
- net SCL_IMU: now also U17.44; no longer U17.43
- net SDA_IMU: now also U17.43; no longer U17.44
Routing:
- net SDA_IMU: track 18.4 -> 32.4 mm, vias 1 -> 0
- net SCL_IMU: track 23.1 -> 31.0 mm
- net INT_IMU: track 10.8 -> 15.3 mm, vias 1 -> 2
- net N$48: track 1.45 -> 5.96 mm, vias 0 -> 1
- net SCLK_LCD: track 19.4 -> 16.6 mm
- net SCS_LCD: track 15.1 -> 12.5 mm
- net N$49: track 6.55 -> 3.86 mm, vias 0 -> 1
- net SI_LCD: track 17.3 -> 14.8 mm
- net GND: track 40.7 -> 43.1 mm, vias 38 -> 36
- net N$2: track 5.14 -> 2.99 mm
- net 3.3V: track 196.6 -> 194.8 mm
- net LED_GREEN: track 26.8 -> 26.1 mm
Other:
- board text added: "The EIR REV1 The Watchmen EECS 473 F15"
